File: kicad/subsheets/microsd.kicad_sch (KiCad schematic)
At the start: 21 parts, among them Q1 FDN340P

Commit message: Annotations
Parts:
- renumbered C54 to C55, C55 to C56, C56 to C57, C57 to C58, R25 to R30, R26 to R31, R27 to R32, R28 to R33, R30 to R34, R31 to R35, R32 to R36, R33 to R37
Connections:
- net PWR renamed SDMMC_PWR
Changed lines of the file:
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@@
 		)
 	)
-	(hierarchical_label "PWR"
+	(hierarchical_label "SDMMC_PWR"
 		(shape input)
 		(at 167.64 33.02 0)
@@
 		(on_board yes)
 		(dnp no)
-		(property "Reference" "R28"
+		(property "Reference" "R33"
 			(at 66.04 37.084 90)
 			(effects
@@
 			(project "srad-camera"
 				(path "/da62c771-e8c9-451f-8df1-ec995aadcb11/f62984d3-000f-4116-a13f-09b83b0ce025"
-					(reference "R28")
+					(reference "R33")
 					(unit 1)
 				)
@@
 		(on_board yes)
 		(dnp no)
-		(property "Reference" "R27"
+		(property "Reference" "R32"
 			(at 66.04 34.544 90)
 			(effects
@@
 			(project "srad-camera"
 				(path "/da62c771-e8c9-451f-8df1-ec995aadcb11/f62984d3-000f-4116-a13f-09b83b0ce025"
-					(reference "R27")
+					(reference "R32")
 					(unit 1)
 				)
@@
 		(on_board yes)
 		(dnp no)
-		(property "Reference" "C57"
+		(property "Reference" "C58"
 			(at 146.812 41.91 0)
 			(effects
@@
 			(project "srad-camera"
 				(path "/da62c771-e8c9-451f-8df1-ec995aadcb11/f62984d3-000f-4116-a13f-09b83b0ce025"
-					(reference "C57")
+					(reference "C58")
 					(unit 1)
 				)
@@
 		(on_board yes)
 		(dnp no)
-		(property "Reference" "C54"
+		(property "Reference" "C55"
 			(at 150.114 21.59 0)
 			(effects
@@
 			(project "srad-camera"
 				(path "/da62c771-e8c9-451f-8df1-ec995aadcb11/f62984d3-000f-4116-a13f-09b83b0ce025"
-					(reference "C54")
+					(reference "C55")
 					(unit 1)
 				)
@@
 		(on_board yes)
 		(dnp no)
-		(property "Reference" "R31"
+		(property "Reference" "R35"
 			(at 66.04 44.704 90)
 			(effects
@@
 			(project "srad-camera"
 				(path "/da62c771-e8c9-451f-8df1-ec995aadcb11/f62984d3-000f-4116-a13f-09b83b0ce025"
-					(reference "R31")
+					(reference "R35")
 					(unit 1)
 				)
@@
 		(dnp no)
 		(fields_autoplaced yes)
-		(property "Reference" "#PWR029"
+		(property "Reference" "#PWR036"
 			(at 106.68 66.04 0)
 			(effects
@@
 			(project "srad-camera"
 				(path "/da62c771-e8c9-451f-8df1-ec995aadcb11/f62984d3-000f-4116-a13f-09b83b0ce025"
-					(reference "#PWR029")
+					(reference "#PWR036")
 					(unit 1)
 				)
@@
 		(on_board yes)
 		(dnp no)
-		(property "Reference" "R26"
+		(property "Reference" "R31"
 			(at 164.846 29.464 90)
 			(effects
@@
 			(project "srad-camera"
 				(path "/da62c771-e8c9-451f-8df1-ec995aadcb11/f62984d3-000f-4116-a13f-09b83b0ce025"
-					(reference "R26")
+					(reference "R31")
 					(unit 1)
 				)
@@
 		(on_board yes)
 		(dnp no)
-		(property "Reference" "R30"
+		(property "Reference" "R34"
 			(at 66.04 42.164 90)
 			(effects
@@
 			(project "srad-camera"
 				(path "/da62c771-e8c9-451f-8df1-ec995aadcb11/f62984d3-000f-4116-a13f-09b83b0ce025"
-					(reference "R30")
+					(reference "R34")
 					(unit 1)
 				)
@@
 		(on_board yes)
 		(dnp no)
-		(property "Reference" "C56"
+		(property "Reference" "C57"
 			(at 141.986 47.244 0)
 			(effects
@@
 			(project "srad-camera"
 				(path "/da62c771-e8c9-451f-8df1-ec995aadcb11/f62984d3-000f-4116-a13f-09b83b0ce025"
-					(reference "C56")
+					(reference "C57")
 					(unit 1)
 				)
@@
 		(on_board yes)
 		(dnp no)
-		(property "Reference" "R32"
+		(property "Reference" "R36"
 			(at 66.04 47.244 90)
 			(effects
@@
 			(project "srad-camera"
 				(path "/da62c771-e8c9-451f-8df1-ec995aadcb11/f62984d3-000f-4116-a13f-09b83b0ce025"
-					(reference "R32")
+					(reference "R36")
 					(unit 1)
 				)
@@
 		(on_board yes)
 		(dnp no)
-		(property "Reference" "C55"
+		(property "Reference" "C56"
 			(at 137.795 47.117 0)
 			(effects
@@
 			(project "srad-camera"
 				(path "/da62c771-e8c9-451f-8df1-ec995aadcb11/f62984d3-000f-4116-a13f-09b83b0ce025"
-					(reference "C55")
+					(reference "C56")
 					(unit 1)
 				)
@@
 		(on_board yes)
 		(dnp no)
-		(property "Reference" "R33"
+		(property "Reference" "R37"
 			(at 66.04 49.784 90)
 			(effects
@@
 			(project "srad-camera"
 				(path "/da62c771-e8c9-451f-8df1-ec995aadcb11/f62984d3-000f-4116-a13f-09b83b0ce025"
-					(reference "R33")
+					(reference "R37")
 					(unit 1)
 				)
@@
 		(on_board yes)
 		(dnp no)
-		(property "Reference" "R25"
+		(property "Reference" "R30"
 			(at 156.464 27.94 0)
 			(effects
@@
 			(project "srad-camera"
 				(path "/da62c771-e8c9-451f-8df1-ec995aadcb11/f62984d3-000f-4116-a13f-09b83b0ce025"
-					(reference "R25")
-					(unit 1)
-				)
+					(reference "R30")
+					(unit 1)
+				)

Commit message: Annotations + minor tweaks
Parts:
- C111: renamed from C56; value 10uF 10V -> 10uF
- R33: renamed from R32; value 33 Ohm 5% -> 33 5%
- R34: renamed from R33; value 33 Ohm 5% -> 33 5%
- R35: renamed from R34; value 33 Ohm 5% -> 33 5%
- R36: renamed from R35; value 33 Ohm 5% -> 33 5%
- R37: renamed from R36; value 33 Ohm 5% -> 33 5%
- R38: renamed from R37; value 33 Ohm 5% -> 33 5%
- renumbered C55 to C110, C57 to C112, C58 to C113, R30 to R31, R31 to R32
Connections:
- net VDD_3V3 renamed VCC_3V3

Commit message: Annotations + minor tweaks
Parts:
- removed C110: 100nF 5%, Capacitor_SMD:C_0201_0603Metric, symbol Device:C_Small
- removed Q1: FDN340P, Package_TO_SOT_SMD:SOT-23, symbol Transistor_FET:FDN340P
- removed R31: 100M, Resistor_SMD:R_0603_1608Metric, symbol Device:R_Small
- removed R32: 10k, Resistor_SMD:R_0603_1608Metric, symbol Device:R_Small
Connections:
- net VCC_3V3: now also C111.2, C112.1, C113.1, D10.2 (A2), MICRO_SD1.4 (VDD)
Other:
- moved on the sheet: C111, C112, C113
