File: kicad/subsheets/rk-soc.kicad_sch (KiCad schematic)
At the start: 1 part, among them U4 RK3566

Commit message: Make sure logic levels are correct between ICs
Other:
- moved on the sheet: U4C, U4D, U4E, U4F, U4G, U4H

Commit message: Annotations
Parts:
- renumbered U4 to U5
Changed lines of the file:
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@@
 		(on_board yes)
 		(dnp no)
-		(property "Reference" "U4"
+		(property "Reference" "U5"
 			(at 179.07 165.1 0)
 			(effects
@@
 			(project "srad-camera"
 				(path "/da62c771-e8c9-451f-8df1-ec995aadcb11/279fc251-45a8-41a3-8fcf-5855d7fe07da"
-					(reference "U4")
+					(reference "U5")
 					(unit 4)
 				)
@@
 		(on_board yes)
 		(dnp no)
-		(property "Reference" "U4"
+		(property "Reference" "U5"
 			(at 48.006 192.532 0)
 			(effects
@@
 			(project "srad-camera"
 				(path "/da62c771-e8c9-451f-8df1-ec995aadcb11/279fc251-45a8-41a3-8fcf-5855d7fe07da"
-					(reference "U4")
+					(reference "U5")
 					(unit 2)
 				)
@@
 		(on_board yes)
 		(dnp no)
-		(property "Reference" "U4"
+		(property "Reference" "U5"
 			(at 177.8 73.66 0)
 			(effects
@@
 			(project "srad-camera"
 				(path "/da62c771-e8c9-451f-8df1-ec995aadcb11/279fc251-45a8-41a3-8fcf-5855d7fe07da"
-					(reference "U4")
+					(reference "U5")
 					(unit 3)
 				)
@@
 		(on_board yes)
 		(dnp no)
-		(property "Reference" "U4"
+		(property "Reference" "U5"
 			(at 306.324 235.712 0)
 			(effects
@@
 			(project "srad-camera"
 				(path "/da62c771-e8c9-451f-8df1-ec995aadcb11/279fc251-45a8-41a3-8fcf-5855d7fe07da"
-					(reference "U4")
+					(reference "U5")
 					(unit 8)
 				)
@@
 		(on_board yes)
 		(dnp no)
-		(property "Reference" "U4"
+		(property "Reference" "U5"
 			(at 47.244 45.466 0)
 			(effects
@@
 			(project "srad-camera"
 				(path "/da62c771-e8c9-451f-8df1-ec995aadcb11/279fc251-45a8-41a3-8fcf-5855d7fe07da"
-					(reference "U4")
+					(reference "U5")
 					(unit 1)
 				)
@@
 		(on_board yes)
 		(dnp no)
-		(property "Reference" "U4"
+		(property "Reference" "U5"
 			(at 173.736 240.03 0)
 			(effects
@@
 			(project "srad-camera"
 				(path "/da62c771-e8c9-451f-8df1-ec995aadcb11/279fc251-45a8-41a3-8fcf-5855d7fe07da"
-					(reference "U4")
+					(reference "U5")
 					(unit 5)
 				)
@@
 		(on_board yes)
 		(dnp no)
-		(property "Reference" "U4"
+		(property "Reference" "U5"
 			(at 306.324 167.894 0)
 			(effects
@@
 			(project "srad-camera"
 				(path "/da62c771-e8c9-451f-8df1-ec995aadcb11/279fc251-45a8-41a3-8fcf-5855d7fe07da"
-					(reference "U4")
+					(reference "U5")
 					(unit 7)
 				)
@@
 		(on_board yes)
 		(dnp no)
-		(property "Reference" "U4"
+		(property "Reference" "U5"
 			(at 309.626 67.31 0)
 			(effects
@@
 			(project "srad-camera"
 				(path "/da62c771-e8c9-451f-8df1-ec995aadcb11/279fc251-45a8-41a3-8fcf-5855d7fe07da"
-					(reference "U4")
+					(reference "U5")
 					(unit 6)
 				)

Commit message: Wire up DDR3L
Parts:
- added C52, C53, C57, C58, C59, C60, C64, C65, C69, C76, C77, C81, C82: 4.7uF, symbol Device:C_Small
- added C54, C55, C56, C61, C63, C66, C68, C70, C72: 22uF, symbol Device:C_Small
- added C62, C67, C71: 10uF, symbol Device:C_Small
- added C73, C74, C75, C78, C79, C80: 100nF, symbol Device:C_Small
- added R29: 240, symbol Device:R_Small
Connections:
- net VDD_CPU: now also U5.1C12 (VDD_CPU_1), U5.1D11 (VDD_CPU_2), U5.1D12 (VDD_CPU_3), U5.1E11 (VDD_CPU_4), U5.1E12 (VDD_CPU_5), U5.1E13 (VDD_CPU_6), U5.1F11 (VDD_CPU_7), U5.1F12 (VDD_CPU_8), U5.1F13 (VDD_CPU_9), U5.1F14 (VDD_CPU_10), U5.1G13 (VDD_CPU_11), C52.1, C53.1, C54.1, C55.1, C56.1
- net VDD_DDR: now also U5.1D5 (DDR_VDDQ_1), U5.1D6 (DDR_VDDQ_2), U5.1D7 (DDR_VDDQ_3), U5.1D8 (DDR_VDDQ_4), U5.1D9 (DDR_VDDQ_5), U5.1E4 (DDR_VDDQ_6), U5.1E6 (DDR_VDDQL_1), U5.1E7 (DDR_VDDQL_2), U5.1E9 (DDR_VDDQL_3), U5.1F4 (DDR_VDDQ_7), U5.1F5 (DDR_VDDQL_4), U5.1G4 (DDR_VDDQ_8), U5.1G5 (DDR_VDDQL_5), C73.2, C74.2, C75.2, C76.2, C77.2, C78.2, C79.2, C80.2, C81.2, C82.2
- net VDD_LOGIC: now also U5.1H10 (VDD_LOGIC_4), U5.1H7 (VDD_LOGIC_1), U5.1H8 (VDD_LOGIC_2), U5.1H9 (VDD_LOGIC_3), U5.1J10 (VDD_LOGIC_6), U5.1J7 (VDD_LOGIC_5), U5.1K10 (VDD_LOGIC_8), U5.1K7 (VDD_LOGIC_7), U5.1L7 (VDD_LOGIC_9), C57.1, C58.1, C59.1, C60.1, C61.1, C62.1, C63.1
- net GND: now reaches U5.1B10 (VSS_30)
- net GND: now also U5.1B11 (VSS_31), U5.1B15 (VSS_32), U5.1B19 (VSS_33), U5.1C14 (VSS_39), U5.1C16 (VSS_40), U5.1C18 (VSS_41), U5.1C4 (VSS_34), U5.1C5 (VSS_35), U5.1C6 (VSS_36), U5.1C8 (VSS_37), U5.1C9 (VSS_38), U5.1D1 (VSS_42), U5.1D10 (VSS_44), U5.1D14 (VSS_45), U5.1D3 (VSS_43), U5.1D4 (DDR_AVSS), U5.1E10 (VSS_48), U5.1E14 (VSS_49), U5.1E15 (VSS_50), U5.1E17 (VSS_51), U5.1E3 (VSS_46), U5.1E8 (VSS_47), U5.1F10 (VSS_56), U5.1F15 (VSS_57), U5.1F16 (VSS_58), U5.1F20 (AVSS1_6), U5.1F6 (VSS_52), U5.1F7 (VSS_53), U5.1F8 (VSS_54), U5.1F9 (VSS_55), U5.1G10 (VSS_64), U5.1G11 (VSS_65), U5.1G12 (VSS_66), U5.1G14 (VSS_67), U5.1G16 (AVSS1_7), U5.1G18 (AVSS1_8), U5.1G19 (AVSS1_9), U5.1G20 (AVSS1_10), U5.1G3 (VSS_59), U5.1G6 (VSS_60), U5.1G7 (VSS_61), U5.1G8 (VSS_62), U5.1G9 (VSS_63), U5.1H1 (VSS_68), U5.1H11 (VSS_71), U5.1H12 (VSS_72), U5.1H13 (VSS_73), U5.1H2 (VSS_69), U5.1H6 (VSS_70), U5.1J1 (VSS_74), U5.1J11 (VSS_78), U5.1J12 (VSS_79), U5.1J13 (VSS_80), U5.1J16 (AVSS1_11), U5.1J18 (AVSS1_12), U5.1J6 (VSS_75), U5.1J8 (VSS_76), U5.1J9 (VSS_77), U5.1K11 (VSS_88), U5.1K12 (VSS_89), U5.1K13 (VSS_90), U5.1K14 (VSS_91), U5.1K15 (VSS_92), U5.1K18 (AVSS1_13), U5.1K2 (VSS_81), U5.1K3 (VSS_82), U5.1K4 (VSS_83), U5.1K5 (VSS_84), U5.1K6 (VSS_85), U5.1K8 (VSS_86), U5.1K9 (VSS_87), U5.1L10 (VSS_95), U5.1L11 (VSS_96), U5.1L12 (VSS_97), U5.1L13 (VSS_98), U5.1L14 (VSS_99), U5.1L15 (VSS_100), U5.1L19 (AVSS1_14), U5.1L3 (VSS_93), U5.1L6 (VSS_94), U5.1M10 (VSS_105), U5.1M11 (VSS_106), U5.1M12 (VSS_107), U5.1M13 (VSS_108), U5.1M14 (VSS_109), U5.1M15 (VSS_110), U5.1M16 (VSS_111), U5.1M17 (VSS_112), U5.1M20 (VSS_113), U5.1M3 (VSS_101), U5.1M4 (VSS_102), U5.1M5 (VSS_103), U5.1M6 (VSS_104), U5.1N11 (AVSS_9), U5.1N12 (AVSS_10), U5.1N3 (VSS_114), U5.1N4 (VSS_115), U5.1N7 (VSS_116), U5.1P1 (VSS_117), U5.1P10 (AVSS_12), U5.1P14 (AVSS_13), U5.1P15 (VSS_121), U5.1P5 (VSS_118), U5.1P6 (VSS_119), U5.1P7 (VSS_120), U5.1P8 (AVSS_11), U5.1R11 (AVSS_16), U5.1R12 (AVSS_17), U5.1R13 (AVSS_18), U5.1R14 (AVSS_19), U5.1R15 (AVSS_20), U5.1R3 (VSS_122), U5.1R4 (VSS_123), U5.1R5 (VSS_124), U5.1R6 (VSS_125), U5.1R7 (VSS_126), U5.1R8 (AVSS_14), U5.1R9 (AVSS_15), U5.1T10 (AVSS_24), U5.1T11 (AVSS_25), U5.1T12 (AVSS_26), U5.1T13 (AVSS_27), U5.1T14 (AVSS_28), U5.1T15 (AVSS_29), U5.1T16 (AVSS_30), U5.1T17 (AVSS_31), U5.1T3 (VSS_127), U5.1T5 (VSS_128), U5.1T7 (AVSS_21), U5.1T8 (AVSS_22), U5.1T9 (AVSS_23), U5.1U12 (AVSS_32), U5.1U13 (AVSS_33), U5.1U15 (AVSS_34), U5.1U17 (AVSS_35), U5.1U2 (VSS_129), U5.1V1 (VSS_130), U5.1V12 (AVSS_37), U5.1V13 (AVSS_38), U5.1V18 (AVSS_39), U5.1V4 (VSS_131), U5.1V7 (AVSS_36), U5.A1 (VSS_1), U5.A2 (VSS_2), U5.A38 (VSS_3), U5.AA2 (VSS_18), U5.AC37 (VSS_24), U5.AD2 (VSS_19), U5.AE37 (VSS_25), U5.AH37 (VSS_26), U5.AL37 (VSS_27), U5.AP13 (AVSS_1), U5.AP16 (AVSS_2), U5.AP19 (AVSS_3), U5.AP2 (VSS_20), U5.AP22 (AVSS_4), U5.AP25 (AVSS_5), U5.AP28 (AVSS_6), U5.AP31 (AVSS_7), U5.AP34 (AVSS_8), U5.AP37 (VSS_28), U5.AP8 (VSS_22), U5.AR1 (VSS_21), U5.AR38 (VSS_29), U5.B1 (VSS_4), U5.B11 (VSS_7), U5.B14 (VSS_8), U5.B18 (VSS_9), U5.B2 (VSS_5), U5.B21 (VSS_10), U5.B28 (VSS_11), U5.B31 (VSS_12), U5.B6 (VSS_6), U5.D2 (VSS_13), U5.E37 (VSS_23), U5.H37 (AVSS1_1), U5.J2 (VSS_14), U5.L2 (VSS_15), U5.L37 (AVSS1_2), U5.P37 (AVSS1_3), U5.U2 (VSS_16), U5.U37 (AVSS1_4), U5.W2 (VSS_17), U5.Y37 (AVSS1_5), C52.2, C53.2, C54.2, C55.2, C56.2, C57.2, C58.2, C59.2, C60.2, C61.2, C62.2, C63.2, C64.2, C65.2, C66.2, C67.2, C68.2, C69.2, C70.2, C71.2, C72.2, C73.1, C74.1, C75.1, C76.1, C77.1, C78.1, C79.1, C80.1, C81.1, C82.1, R29.1
- net RASn: now reaches U5.1A1 (AC16)
- net CASn: now reaches U5.1A2 (AC17)
- net A10: now reaches U5.1A3 (AC10)
- net WEn: now reaches U5.1A4 (AC20)
- net ODT0: now reaches U5.1A5 (AC27)
- net A12: now reaches U5.1A6 (AC19)
- net BA2: now reaches U5.1B3 (AC12)
- net CSn0: now reaches U5.1B5 (AC28)
- net BA1: now reaches U5.1B6 (AC4)
- net A1: now reaches U5.1B7 (AC18)
- net A0: now reaches U5.1C1 (AC15)
- net BA0: now reaches U5.1C2 (AC21)
- net A3: now reaches U5.1C3 (AC3)
- net RESETn: now reaches U5.1C7 (AC29)
- net A2: now reaches U5.1D2 (AC1)
- net DQ7: now reaches U5.1E1 (DDR_DQ7_A)
- net DM_A0: now reaches U5.1E2 (DDR_DM0_A)
- net DQ14: now reaches U5.1F1 (DDR_DQ14_A)
- net DQ13: now reaches U5.1F2 (DDR_DQ13_A)
- net at U5.1F3 (DDR_RZQ): now also R29.2
- net DM_A1: now reaches U5.1G1 (DDR_DM1_A)
- net DQ15: now reaches U5.1G2 (DDR_DQ15_A)
- net DDR_VREFOUT: now reaches U5.1H3 (DDR_VREFOUT)
- net A8: now reaches U5.A10 (AC7)
- net CK_P: now reaches U5.A5 (AC23)
- net A9: now reaches U5.A7 (AC0)
- net A14: now reaches U5.A9 (AC13)
- net CKE: now reaches U5.B4 (AC22)
- net CK_N: now reaches U5.B5 (AC24)
- net A5: now reaches U5.B7 (AC9)
- net A11: now reaches U5.B8 (AC5)
- net A13: now reaches U5.B9 (AC6)
- net A4: now reaches U5.C1 (AC2)
- net A7: now reaches U5.C2 (AC11)
- net DQ3: now reaches U5.E1 (DDR_DQ3_A)
- net A6: now reaches U5.E2 (AC8)
- net DQ2: now reaches U5.F1 (DDR_DQ2_A)
- net DQ1: now reaches U5.F2 (DDR_DQ1_A)
- net DQ0: now reaches U5.G2 (DDR_DQ0_A)
- net DQS_N0: now reaches U5.H1 (DDR_DQS0N_A)
- net DQS_P0: now reaches U5.H2 (DDR_DQS0P_A)
- net DQ5: now reaches U5.K1 (DDR_DQ5_A)
- net DQ6: now reaches U5.K2 (DDR_DQ6_A)
- net DQ12: now reaches U5.M1 (DDR_DQ12_A)
- net DQ4: now reaches U5.M2 (DDR_DQ4_A)
- net DQS_P1: now reaches U5.N1 (DDR_DQS1P_A)
- net DQS_N1: now reaches U5.N2 (DDR_DQS1N_A)
- net DQ8: now reaches U5.P2 (DDR_DQ8_A)
- net DQ9: now reaches U5.R1 (DDR_DQ9_A)
- net DQ10: now reaches U5.R2 (DDR_DQ10_A)
- net DQ11: now reaches U5.T2 (DDR_DQ11_A)
- net VDD_GPU_NPU: now reaches U5.1G15 (VDD_NPU_1)
- net VDD_GPU_NPU: now also U5.1H14 (VDD_NPU_2), U5.1H15 (VDD_NPU_3), U5.1J14 (VDD_NPU_4), U5.1J15 (VDD_NPU_5), U5.1L8 (VDD_GPU_1), U5.1L9 (VDD_GPU_2), U5.1M7 (VDD_GPU_3), U5.1M8 (VDD_GPU_4), U5.1M9 (VDD_GPU_5), C64.1, C65.1, C66.1, C67.1, C68.1, C69.1, C70.1, C71.1, C72.1
- no-connect marks 0 -> 25
Other:
- moved on the sheet: U5A, U5B, U5C, U5D, U5E, U5F, U5G, U5H

Commit message: Finished wiring RK3566, DDR3L
Parts:
- added C110, C114, C115, C116, C117, C118, C121, C122, C123, C124, C125, C126, C128, C129, C130, C131, C132, C134, C135, C136, C137, C140, C142, C144, C146, C147, C148, C149, C150, C151, C152, C153, C155: 100nF, symbol Device:C_Small
- added C119, C120: 18pF, symbol Device:C_Small
- added C133, C138, C139, C141, C143, C145: 1uF, symbol Device:C_Small
- added C154: 1nF, symbol Device:C_Small
- added HSE2: 24MHz, symbol Device:Crystal_GND24
- added R31, R41, R44, R48: 0R, symbol Device:R_Small
- added R39, R40, R42, R43, R51: 1R, symbol Device:R_Small
- added R45: 10k, symbol Device:R_Small
- added R47, R50: 22R, symbol Device:R_Small
- added R49: 1M, symbol Device:R_Small
- added R53: 100R, symbol Device:R_Small
- R29: value 240 -> 120R 1%
Connections:
- net GND: now also U5.1J5 (SYSPLL_AVSS), U5.1N17 (PMUPLL_AVSS), C110.1, C114.1, C115.1, C116.1, C117.1, C118.1, C119.2, C120.2, C121.1, C122.1, C123.1, C124.1, C125.1, C126.1, C128.1, C129.1, C130.1, C131.1, C132.1, C133.1, C134.1, C135.1, C136.1, C137.1, C138.1, C139.1, C140.1, C141.2, C142.2, C143.2, C144.2, C145.1, C146.1, C147.1, C148.1, C149.1, C150.1, C151.1, C152.1, C153.1, C154.1, C155.2, HSE2.2, HSE2.4, R48.2, R53.2
- net RK_RX: now also U5.1T19 (GPIO0_C0_d)
- net RK_TX: now also U5.1R18 (GPIO0_C1_d)
- net USB_DM: now also U5.R38 (USB_OTG0_DM)
- net USB_DP: now also U5.R37 (USB_OTG0_DP)
- net VCCA_1V8: now also U5.1D15 (OTP_VCC1V8), U5.1D16 (SARADC_AVDD_1V8), U5.1H4 (SYSPLL_AVDD_1V8), U5.1K17 (MULTI_PHY_AVDD_1V8), C124.2, C143.1, C144.1, C153.2, R40.1, R42.1, R45.2
- net VCCA_1V8_IMG: now also U5.1P13 (HDMI_TX_AVDD_1V8), C145.2, C151.2, R51.2
- net VCCA_1V8_PMU: now also U5.1E16 (VCCIO4), U5.1N18 (PMUPLL_AVDD_1V8), C137.2, C139.2, C140.2
- net VCC_1V8: now also U5.1C13 (VCCIO2), C134.2
- net VCC_3V3: now also U5.1D13 (VCCIO1), U5.1L4 (VCCIO6_1), U5.1L5 (VCCIO6_2), U5.1N5 (VCCIO5_1), U5.1N6 (VCCIO5_2), U5.1N8 (VCCIO7), C126.2, C130.2, C135.2, C136.2, R41.1, R44.1
- net VCC_3V3_PMU: now also U5.1N15 (PMUIO2), U5.1P16 (PMUIO1), C128.2, C131.2
- net VDDA_0V9: now also U5.1H5 (SYSPLL_AVDD_0V9), U5.1K16 (MULTI_PHY_AVDD_0V9), C125.2, C141.1, C142.1, R39.1, R43.1
- net VDDA_0V9_IMG: now also U5.1N10 (MIPI_DSI_TX1_AVDD_0V9), U5.1N13 (HDMI_TX_AVDD_0V9_2), U5.1N14 (HDMI_TX_AVDD_0V9_1), U5.1N9 (MIPI_CSI_RX_AVDD_0V9), U5.1P11 (MIPI_DSI_TX0/LVDS_TX0_AVDD_0V9), C114.2, C146.2, C150.2, C152.2
- net VDDA_0V9_PMU: now also U5.1N16 (PMU_VDD_LOGIC_0V9), U5.1P17 (PMUPLL_AVDD_0V9), C132.2, C133.2, C138.2, C147.2
- net at U5.1M18 (TVSS): now also R48.1
- net PMIC_SLEEP: now reaches U5.1P19 (GPIO0_A2_d)
- net TSADC_SHUT: now reaches U5.1R20 (GPIO0_A1_z)
- net TSADC_SHUT: now also R31.1
- net PMIC_CLK32: now reaches U5.1T20 (GPIO0_B0_u)
- net XIN: now reaches U5.AD37 (XIN24M)
- net XIN: now also C120.1, HSE2.1, R49.2
- net XOUT: now reaches U5.AD38 (XOUT24M)
- net XOUT: now also R49.1, R50.1
- net at U5.AF37 (GPIO0_A4_u): now also R53.1
- net PMIC_RESET: now reaches U5.AG38 (nPOR_u)
- net PMIC_RESET: now also C110.2, R31.2
- net at U5.1H16 (USB_AVDD1_1V8): now also C117.2, R40.2
- net at U5.1H18 (USB_AVDD1_3V3): now also C118.2, R41.2
- net at U5.1J17 (USB_AVDD1_0V9): now also C116.2, R39.2
- net at U5.1J2 (USB_AVDD2_3V3): now also C123.2, R44.2
- net at U5.1J3 (USB_AVDD2_1V8): now also C122.2, R42.2
- net at U5.1J4 (USB_AVDD2_0V9): now also C121.2, R43.2
- net USB_DET: now reaches U5.T38 (USB_OTG0_VBUSDET)
- net USB_DET: now also C155.1
- net D1: now reaches U5.1A14 (GPIO1_A6_d)
- net CMD: now reaches U5.1E19 (GPIO2_A1_u)
- net VCCIO_3V3_SD: now reaches U5.1F17 (VCCIO3)
- net VCCIO_3V3_SD: now also C129.2
- net D3: now reaches U5.1F18 (GPIO2_A0_u)
- net D0: now reaches U5.B24 (GPIO1_A5_d)
- net D2: now reaches U5.B25 (GPIO1_A7_d)
- net at U5.G38 (GPIO2_A2_d): now also R47.2
- net MIPI_AVDD_1V8: now reaches U5.1P12 (MIPI_DSI_TX0/LVDS_TX0_AVDD_1V8)
- net MIPI_AVDD_1V8: now also U5.1P9 (MIPI_CSI_RX_AVDD_1V8), U5.1R10 (MIPI_DSI_TX1_AVDD_1V8), C115.2, C148.2, C149.2, R51.1
- net MIPI_CN: now reaches U5.1U9 (MIPI_CSI_RX_CLK0N)
- net MIPI_CP: now reaches U5.1V9 (MIPI_CSI_RX_CLK0P)
- net MIPI_DN3: now reaches U5.AP14 (MIPI_CSI_RX_D3N)
- net MIPI_DP2: now reaches U5.AP15 (MIPI_CSI_RX_D2P)
- net MIPI_DN1: now reaches U5.AP17 (MIPI_CSI_RX_D1N)
- net MIPI_DP0: now reaches U5.AP18 (MIPI_CSI_RX_D0P)
- net MIPI_DP3: now reaches U5.AR14 (MIPI_CSI_RX_D3P)
- net MIPI_DN2: now reaches U5.AR15 (MIPI_CSI_RX_D2N)
- net MIPI_DP1: now reaches U5.AR17 (MIPI_CSI_RX_D1P)
- net MIPI_DN0: now reaches U5.AR18 (MIPI_CSI_RX_D0N)
- net at U5.1D17 (SARADC_VIN0): now also C154.2, R45.1
- net CAM_GPIO0: now reaches U5.1T2 (GPIO3_C6_d)
- net CAM_GPIO1: now reaches U5.AB2 (GPIO4_C0_d)
- net CAM_SCL: now reaches U5.AD1 (GPIO4_B5_d)
- net CAM_SDA: now reaches U5.AF1 (GPIO4_B4_d)
- new net: C119.1, HSE2.3, R50.2
- new net CLK: R47.1
- no-connect marks 25 -> 215
Other:
- note added: "CIF_CLKOUT"
- note added: "Caps close to package"
- note added: "Caps under package"
- note added: "I2C2"
- note added: "SDMMC0_DET"
- note added: "UART0_RX"
- note added: "UART0_TX"
- moved on the sheet: C52, C53, C54, C55, C56, C57, C58, C59, C60, C61, C62, C63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

Commit message: Change all sheets to A4, name sheets, split RK3566 into hierarchy
Parts:
- removed C110, C114, C115, C116, C117, C118, C121, C122, C123, C124, C125, C126, C128, C129, C130, C131, C132, C134, C135, C136, C137, C140, C142, C144, C146, C147, C148, C149, C150, C151, C152, C153, C155, C73, C74, C75, C78, C79, C80: 100nF, symbol Device:C_Small
- removed C119, C120: 18pF, symbol Device:C_Small
- removed C133, C138, C139, C141, C143, C145: 1uF, symbol Device:C_Small
- removed C154: 1nF, symbol Device:C_Small
- removed C76, C77, C81, C82: 4.7uF, symbol Device:C_Small
- removed HSE2: 24MHz, symbol Device:Crystal_GND24
- removed R29: 120R 1%, symbol Device:R_Small
- removed R31, R41, R44, R48: 0R, symbol Device:R_Small
- removed R39, R40, R42, R43, R51: 1R, symbol Device:R_Small
- removed R45: 10k, symbol Device:R_Small
- removed R47, R50: 22R, symbol Device:R_Small
- removed R49: 1M, symbol Device:R_Small
- removed R53: 100R, symbol Device:R_Small
- removed unit 4 of U5
- removed unit 3 of U5
- removed unit 8 of U5
- removed unit 5 of U5
- removed unit 7 of U5
- removed unit 6 of U5
Connections:
- no-connect marks 215 -> 0
Other:
- added sheet DDR PHY (rk-domains/ddr-phy.kicad_sch)
- added sheet MIPI CSI-DSI, HDMI (rk-domains/mipi-csi-dsi-hdmi.kicad_sch)
- added sheet PMUIO 1-2, OSC (rk-domains/pmuio1-2-osc.kicad_sch)
- added sheet USB AVDD (rk-domains/usb-avdd.kicad_sch)
- added sheet VCCIO 1-4 (rk-domains/vccio1-4.kicad_sch)
- added sheet VCCIO 5-7 (rk-domains/vccio5-7.kicad_sch)
- note removed: "CIF_CLKOUT"
- note removed: "I2C2"
- note removed: "SDMMC0_DET"
- note removed: "UART0_RX"
- note removed: "UART0_TX"
- moved on the sheet: C52, C53, C54, C55, C56, C57, C58, C59, C60, C61, C62, C63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
