File: kicad/subsheets/rk-soc.kicad_sch (KiCad schematic)
At the start: 22 parts, among them U5 RK3566

Commit message: Mark as R1.0
Parts:
- renumbered C56 to C53, C55 to C54, C54 to C55, C53 to C56, C52 to C57, C63 to C58, C62 to C59, C61 to C60, C60 to C61, C59 to C62, C58 to C63, C57 to C64, C68 to C65, C67 to C66, C66 to C67, C65 to C68, C64 to C69, C72 to C70, C70 to C72, C69 to C73
Other:
- company: (none) -> UVic Rocketry
- title: (none) -> RK3566 SoC
Changed lines of the file:
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@@
 	(generator_version "9.0")
 	(paper "A4")
+	(title_block
+		(title "RK3566 SoC")
+		(date "2025-11-23")
+		(rev "1.0")
+		(company "UVic Rocketry")
+		(comment 1 "Author: Eric Handley")
+	)
 	(text "Caps close\nto package"
 		(exclude_from_sim no)
@@
 		(dnp no)
 		(fields_autoplaced yes)
-		(property "Reference" "C63"
+		(property "Reference" "C58"
 			(at 73.66 66.04 0)
 			(effects
@@
 			(project "srad-camera"
 				(path "/da62c771-e8c9-451f-8df1-ec995aadcb11/279fc251-45a8-41a3-8fcf-5855d7fe07da"
-					(reference "C63")
+					(reference "C58")
 					(unit 1)
 				)
@@
 		(dnp no)
 		(fields_autoplaced yes)
-		(property "Reference" "#PWR047"
+		(property "Reference" "#PWR054"
 			(at 113.03 125.73 0)
 			(effects
@@
 			(project "srad-camera"
 				(path "/da62c771-e8c9-451f-8df1-ec995aadcb11/279fc251-45a8-41a3-8fcf-5855d7fe07da"
-					(reference "#PWR047")
+					(reference "#PWR054")
 					(unit 1)
 				)
@@
 		(dnp no)
 		(fields_autoplaced yes)
-		(property "Reference" "C56"
+		(property "Reference" "C53"
 			(at 73.66 35.56 0)
 			(effects
@@
 			(project "srad-camera"
 				(path "/da62c771-e8c9-451f-8df1-ec995aadcb11/279fc251-45a8-41a3-8fcf-5855d7fe07da"
-					(reference "C56")
+					(reference "C53")
 					(unit 1)
 				)
@@
 		(dnp no)
 		(fields_autoplaced yes)
-		(property "Reference" "#PWR044"
+		(property "Reference" "#PWR050"
 			(at 73.66 85.09 0)
 			(effects
@@
 			(project "srad-camera"
 				(path "/da62c771-e8c9-451f-8df1-ec995aadcb11/279fc251-45a8-41a3-8fcf-5855d7fe07da"
-					(reference "#PWR044")
+					(reference "#PWR050")
 					(unit 1)
 				)
@@
 		(dnp no)
 		(fields_autoplaced yes)
-		(property "Reference" "C57"
+		(property "Reference" "C64"
 			(at 119.38 66.04 0)
 			(effects
@@
 			(project "srad-camera"
 				(path "/da62c771-e8c9-451f-8df1-ec995aadcb11/279fc251-45a8-41a3-8fcf-5855d7fe07da"
-					(reference "C57")
+					(reference "C64")
 					(unit 1)
 				)
@@
 		(dnp no)
 		(fields_autoplaced yes)
-		(property "Reference" "#PWR048"
+		(property "Reference" "#PWR053"
 			(at 64.77 125.73 0)
 			(effects
@@
 			(project "srad-camera"
 				(path "/da62c771-e8c9-451f-8df1-ec995aadcb11/279fc251-45a8-41a3-8fcf-5855d7fe07da"
-					(reference "#PWR048")
+					(reference "#PWR053")
 					(unit 1)
 				)
@@
 		(dnp no)
 		(fields_autoplaced yes)
-		(property "Reference" "C59"
+		(property "Reference" "C62"
 			(at 106.68 66.04 0)
 			(effects
@@
 			(project "srad-camera"
 				(path "/da62c771-e8c9-451f-8df1-ec995aadcb11/279fc251-45a8-41a3-8fcf-5855d7fe07da"
-					(reference "C59")
+					(reference "C62")
 					(unit 1)
 				)
@@
 		(dnp no)
 		(fields_autoplaced yes)
-		(property "Reference" "C69"
+		(property "Reference" "C73"
 			(at 119.38 106.68 0)
 			(effects
@@
 			(project "srad-camera"
 				(path "/da62c771-e8c9-451f-8df1-ec995aadcb11/279fc251-45a8-41a3-8fcf-5855d7fe07da"
-					(reference "C69")
+					(reference "C73")
 					(unit 1)
 				)
@@
 		(dnp no)
 		(fields_autoplaced yes)
-		(property "Reference" "C67"
+		(property "Reference" "C66"
 			(at 80.01 91.44 0)
 			(effects
@@
 			(project "srad-camera"
 				(path "/da62c771-e8c9-451f-8df1-ec995aadcb11/279fc251-45a8-41a3-8fcf-5855d7fe07da"
-					(reference "C67")
+					(reference "C66")
 					(unit 1)
 				)
@@
 		(dnp no)
 		(fields_autoplaced yes)
-		(property "Reference" "C54"
+		(property "Reference" "C55"
 			(at 106.68 35.56 0)
 			(effects
@@
 			(project "srad-camera"
 				(path "/da62c771-e8c9-451f-8df1-ec995aadcb11/279fc251-45a8-41a3-8fcf-5855d7fe07da"
-					(reference "C54")
+					(reference "C55")
 					(unit 1)
 				)
@@
 		(dnp no)
 		(fields_autoplaced yes)
-		(property "Reference" "C52"
+		(property "Reference" "C57"
 			(at 119.38 35.56 0)
 			(effects
@@
 			(project ""
 				(path "/da62c771-e8c9-451f-8df1-ec995aadcb11/279fc251-45a8-41a3-8fcf-5855d7fe07da"
-					(reference "C52")
+					(reference "C57")
 					(unit 1)
 				)
@@
 		(dnp no)
 		(fields_autoplaced yes)
-		(property "Reference" "C64"
+		(property "Reference" "C69"
 			(at 119.38 91.44 0)
 			(effects
@@
 			(project "srad-camera"
 				(path "/da62c771-e8c9-451f-8df1-ec995aadcb11/279fc251-45a8-41a3-8fcf-5855d7fe07da"
-					(reference "C64")
+					(reference "C69")
 					(unit 1)
 				)
@@
 		(dnp no)
 		(fields_autoplaced yes)
-		(property "Reference" "C58"
+		(property "Reference" "C63"
 			(at 113.03 66.04 0)
 			(effects
@@
 			(project "srad-camera"
 				(path "/da62c771-e8c9-451f-8df1-ec995aadcb11/279fc251-45a8-41a3-8fcf-5855d7fe07da"
-					(reference "C58")
+					(reference "C63")
 					(unit 1)
 				)
@@
 		(dnp no)
 		(fields_autoplaced yes)
-		(property "Reference" "#PWR043"
+		(property "Reference" "#PWR051"
 			(at 93.98 85.09 0)
 			(effects
@@
 			(project "srad-camera"
 				(path "/da62c771-e8c9-451f-8df1-ec995aadcb11/279fc251-45a8-41a3-8fcf-5855d7fe07da"
-					(reference "#PWR043")
+					(reference "#PWR051")
 					(unit 1)
 				)
@@
 		(dnp no)
 		(fields_autoplaced yes)
-		(property "Reference" "C55"
+		(property "Reference" "C54"
 			(at 80.01 35.56 0)
 			(effects
@@
 			(project "srad-camera"
 				(path "/da62c771-e8c9-451f-8df1-ec995aadcb11/279fc251-45a8-41a3-8fcf-5855d7fe07da"
-					(reference "C55")
+					(reference "C54")
 					(unit 1)
 				)
@@
 		(on_board yes)
 		(dnp no)
-		(property "Reference" "#PWR052"
+		(property "Reference" "#PWR055"
 			(at 125.73 139.7 0)
 			(effects
@@
 			(project "srad-camera"
 				(path "/da62c771-e8c9-451f-8df1-ec995aadcb11/279fc251-45a8-41a3-8fcf-5855d7fe07da"
-					(reference "#PWR052")
+					(reference "#PWR055")
 					(unit 1)
 				)
@@
 		(dnp no)
 		(fields_autoplaced yes)
-		(property "Reference" "C60"
+		(property "Reference" "C61"
 			(at 100.33 66.04 0)
 			(effects
@@
 			(project "srad-camera"
 				(path "/da62c771-e8c9-451f-8df1-ec995aadcb11/279fc251-45a8-41a3-8fcf-5855d7fe07da"
-					(reference "C60")
+					(reference "C61")
 					(unit 1)
 				)
@@
 		(dnp no)
 		(fields_autoplaced yes)
-		(property "Reference" "C61"
+		(property "Reference" "C60"
 			(at 93.98 66.04 0)
 			(effects
@@
 			(project "srad-camera"
 				(path "/da62c771-e8c9-451f-8df1-ec995aadcb11/279fc251-45a8-41a3-8fcf-5855d7fe07da"
-					(reference "C61")
+					(reference "C60")
 					(unit 1)
 				)
@@
 		(dnp no)
 		(fields_autoplaced yes)
-		(property "Reference" "C62"
+		(property "Reference" "C59"
 			(at 80.01 66.04 0)
 			(effects
@@
 			(project "srad-camera"
 				(path "/da62c771-e8c9-451f-8df1-ec995aadcb11/279fc251-45a8-41a3-8fcf-5855d7fe07da"
-					(reference "C62")
+					(reference "C59")
 					(unit 1)
 				)
@@
 		(dnp no)
 		(fields_autoplaced yes)
-		(property "Reference" "#PWR041"
+		(property "Reference" "#PWR049"
 			(at 106.68 54.61 0)
 			(effects
@@
 			(project "srad-camera"
 				(path "/da62c771-e8c9-451f-8df1-ec995aadcb11/279fc251-45a8-41a3-8fcf-5855d7fe07da"
-					(reference "#PWR041")
+					(reference "#PWR049")
 					(unit 1)
 				)
@@
 		(dnp no)
 		(fields_autoplaced yes)
-		(property "Reference" "C72"
+		(property "Reference" "C70"
 			(at 73.66 106.68 0)
 			(effects
@@
 			(project "srad-camera"
 				(path "/da62c771-e8c9-451f-8df1-ec995aadcb11/279fc251-45a8-41a3-8fcf-5855d7fe07da"
-					(reference "C72")
+					(reference "C70")
 					(unit 1)
 				)
@@
 		(dnp no)
 		(fields_autoplaced yes)
-		(property "Reference" "C53"
+		(property "Reference" "C56"
 			(at 113.03 35.56 0)
 			(effects
@@
 			(project "srad-camera"
 				(path "/da62c771-e8c9-451f-8df1-ec995aadcb11/279fc251-45a8-41a3-8fcf-5855d7fe07da"
-					(reference "C53")
+					(reference "C56")
 					(unit 1)
 				)
@@
 		(dnp no)
 		(fields_autoplaced yes)
-		(property "Reference" "#PWR042"
+		(property "Reference" "#PWR048"
 			(at 73.66 54.61 0)
 			(effects
@@
 			(project "srad-camera"
 				(path "/da62c771-e8c9-451f-8df1-ec995aadcb11/279fc251-45a8-41a3-8fcf-5855d7fe07da"
-					(reference "#PWR042")
+					(reference "#PWR048")
 					(unit 1)
 				)
@@
 		(dnp no)
 		(fields_autoplaced yes)
-		(property "Reference" "#PWR045"
+		(property "Reference" "#PWR052"
 			(at 106.68 110.49 0)
 			(effects
@@
 			(project "srad-camera"
 				(path "/da62c771-e8c9-451f-8df1-ec995aadcb11/279fc251-45a8-41a3-8fcf-5855d7fe07da"
-					(reference "#PWR045")
+					(reference "#PWR052")
 					(unit 1)
 				)
@@
 		(dnp no)
 		(fields_autoplaced yes)
-		(property "Reference" "C65"
+		(property "Reference" "C68"
 			(at 113.03 91.44 0)
 			(effects
@@
 			(project "srad-camera"
 				(path "/da62c771-e8c9-451f-8df1-ec995aadcb11/279fc251-45a8-41a3-8fcf-5855d7fe07da"
-					(reference "C65")
+					(reference "C68")
 					(unit 1)
 				)
@@
 		(dnp no)
 		(fields_autoplaced yes)
-		(property "Reference" "C70"
+		(property "Reference" "C72"
 			(at 113.03 106.68 0)
 			(effects
@@
 			(project "srad-camera"
 				(path "/da62c771-e8c9-451f-8df1-ec995aadcb11/279fc251-45a8-41a3-8fcf-5855d7fe07da"
-					(reference "C70")
+					(reference "C72")
 					(unit 1)
 				)
@@
 		(dnp no)
 		(fields_autoplaced yes)
-		(property "Reference" "C66"
+		(property "Reference" "C67"
 			(at 106.68 91.44 0)
 			(effects
@@
 			(project "srad-camera"
 				(path "/da62c771-e8c9-451f-8df1-ec995aadcb11/279fc251-45a8-41a3-8fcf-5855d7fe07da"
-					(reference "C66")
+					(reference "C67")
 					(unit 1)
 				)
@@
 		(dnp no)
 		(fields_autoplaced yes)
-		(property "Reference" "C68"
+		(property "Reference" "C65"
 			(at 73.66 91.44 0)
 			(effects
@@
 			(project "srad-camera"
 				(path "/da62c771-e8c9-451f-8df1-ec995aadcb11/279fc251-45a8-41a3-8fcf-5855d7fe07da"
-					(reference "C68")
+					(reference "C65")
 					(unit 1)
 				)

Commit message: Indicate proper feedback trace from SoC
Parts:
- renumbered C53 to C66, C54 to C67, C55 to C68, C56 to C69, C57 to C70, C58 to C71, C59 to C72, C60 to C73, C61 to C74, C62 to C75, C63 to C76, C64 to C77, C65 to C78, C66 to C79, C67 to C80, C68 to C81, C69 to C82, C70 to C83, C71 to C84, C72 to C85, C73 to C86
Other:
- note added: "U5 RK3566"
- moved on the sheet: C66, C67, C68, C69, C70, C71, C72, C73, C74, C75, C76, C77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

Commit message: Minor tweaks + annotations
Changed lines of the file:
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@@
 	)
 	(junction
-		(at 69.85 120.65)
-		(diameter 0)
-		(color 0 0 0 0)
-	)
-	(junction
 		(at 106.68 41.91)
 		(diameter 0)
@@
 	)
 	(junction
-		(at 67.31 97.79)
-		(diameter 0)
-		(color 0 0 0 0)
-	)
-	(junction
 		(at 113.03 105.41)
 		(diameter 0)
@@
 	(wire
 		(pts
-			(xy 69.85 121.92) (xy 69.85 120.65)
+			(xy 67.31 121.92) (xy 67.31 120.65)
 		)
 		(stroke
@@
 	(wire
 		(pts
-			(xy 69.85 105.41) (xy 69.85 120.65)
-		)
-		(stroke
-			(width 0)
-			(type default)
-		)
-	)
-	(wire
-		(pts
 			(xy 171.45 72.39) (xy 167.64 72.39)
 		)
@@
 	(wire
 		(pts
-			(xy 69.85 105.41) (xy 73.66 105.41)
+			(xy 67.31 105.41) (xy 73.66 105.41)
 		)
 		(stroke
@@
 		)
 	)
+	(polyline
+		(pts
+			(xy 87.63 129.54) (xy 104.14 129.54)
+		)
+		(stroke
+			(width 0.25)
+			(type dash)
+			(color 0 0 255 1)
+		)
+	)
 	(wire
 		(pts
@@
 	(wire
 		(pts
-			(xy 73.66 120.65) (xy 69.85 120.65)
+			(xy 73.66 120.65) (xy 67.31 120.65)
 		)
 		(stroke
@@
 	(wire
 		(pts
+			(xy 63.5 113.03) (xy 73.66 113.03)
+		)
+		(stroke
+			(width 0)
+			(type default)
+		)
+	)
+	(wire
+		(pts
 			(xy 167.64 52.07) (xy 196.85 52.07)
 		)
@@
 	(wire
 		(pts
-			(xy 67.31 97.79) (xy 64.77 97.79)
+			(xy 64.77 97.79) (xy 73.66 97.79)
 		)
 		(stroke
@@
 	(wire
 		(pts
-			(xy 67.31 97.79) (xy 67.31 113.03)
-		)
-		(stroke
-			(width 0)
-			(type default)
-		)
-	)
-	(wire
-		(pts
 			(xy 113.03 80.01) (xy 113.03 78.74)
 		)
@@
 		)
 	)
-	(polyline
-		(pts
-			(xy 102.87 129.54) (xy 87.63 129.54)
-		)
-		(stroke
-			(width 0.25)
-			(type dash)
-			(color 0 0 255 1)
-		)
-	)
 	(wire
 		(pts
@@
 	(wire
 		(pts
-			(xy 67.31 97.79) (xy 73.66 97.79)
-		)
-		(stroke
-			(width 0)
-			(type default)
-		)
-	)
-	(wire
-		(pts
 			(xy 124.46 41.91) (xy 127 41.91)
 		)
@@
 	(wire
 		(pts
+			(xy 67.31 105.41) (xy 67.31 106.68)
+		)
+		(stroke
+			(width 0)
+			(type default)
+		)
+	)
+	(wire
+		(pts
 			(xy 73.66 113.03) (xy 80.01 113.03)
 		)
@@
 	(wire
 		(pts
-			(xy 67.31 113.03) (xy 73.66 113.03)
-		)
-		(stroke
-			(width 0)
-			(type default)
-		)
-	)
-	(wire
-		(pts
 			(xy 73.66 120.65) (xy 73.66 119.38)
 		)
@@
 		)
 	)
+	(hierarchical_label "VDD_GPU_NPU"
+		(shape input)
+		(at 63.5 113.03 180)
+		(effects
+			(font
+				(size 1.27 1.27)
+			)
+			(justify right)
+		)
+	)
 	(hierarchical_label "VCCA_1V8"
 		(shape input)
@@
 	(symbol
 		(lib_id "power:GND")
-		(at 69.85 121.92 0)
+		(at 67.31 121.92 0)
 		(mirror y)
 		(unit 1)
@@
 		(fields_autoplaced yes)
 		(property "Reference" "#PWR063"
-			(at 69.85 128.27 0)
+			(at 67.31 128.27 0)
 			(effects
 				(font
@@
 		)
 		(property "Value" "GND"
-			(at 69.85 125.984 0)
+			(at 67.31 125.984 0)
 			(effects
 				(font
@@
 		)
 		(property "Footprint" ""
-			(at 69.85 121.92 0)
+			(at 67.31 121.92 0)
 			(effects
 				(font
@@
 		)
 		(property "Datasheet" ""
-			(at 69.85 121.92 0)
+			(at 67.31 121.92 0)
 			(effects
 				(font
@@
 		)
 		(property "Description" "Power symbol creates a global label with name \"GND\" , ground"
-			(at 69.85 121.92 0)
+			(at 67.31 121.92 0)
 			(effects
 				(font
@@
 					(unit 1)
 				)
+			)
+		)
+	)
+	(symbol
+		(lib_id "power:GND")
+		(at 67.31 106.68 0)
+		(mirror y)
+		(unit 1)
+		(exclude_from_sim no)
+		(in_bom yes)
+		(on_board yes)
+		(dnp no)
+		(fields_autoplaced yes)
+		(property "Reference" "#PWR0108"
+			(at 67.31 113.03 0)
+			(effects
+				(font
+					(size 1.27 1.27)
+				)
+				(hide yes)
+			)
+		)
+		(property "Value" "GND"
+			(at 67.31 110.744 0)
+			(effects
+				(font
+					(size 1.27 1.27)
+				)
+			)
+		)
+		(property "Footprint" ""
+			(at 67.31 106.68 0)
+			(effects
+				(font
+					(size 1.27 1.27)
+				)
+				(hide yes)
+			)
+		)
+		(property "Datasheet" ""
+			(at 67.31 106.68 0)
+			(effects
+				(font
+					(size 1.27 1.27)
+				)
+				(hide yes)
+			)
+		)
+		(property "Description" "Power symbol creates a global label with name \"GND\" , ground"
+			(at 67.31 106.68 0)
+			(effects
+				(font
+					(size 1.27 1.27)
+				)
+				(hide yes)
+			)
+		)
+		(pin "1"
+		)
+		(instances
+			(project "srad-camera"
+				(path "/da62c771-e8c9-451f-8df1-ec995aadcb11/279fc251-45a8-41a3-8fcf-5855d7fe07da"
+					(reference "#PWR0108")
+					(unit 1)
+				)

Commit message: Start on PCB design
Parts:
- added NT4, NT5: NetTie_2, symbol Device:NetTie_2
- C64: renamed from C66; footprint (none) -> Capacitor_SMD:C_1206_3216Metric; LCSC PART NAME (none) -> C12891
- C65: renamed from C67; footprint (none) -> Capacitor_SMD:C_1206_3216Metric; LCSC PART NAME (none) -> C12891
- C66: renamed from C68; footprint (none) -> Capacitor_SMD:C_1206_3216Metric; LCSC PART NAME (none) -> C12891
- C67: renamed from C69; footprint (none) -> Capacitor_SMD:C_0805_2012Metric; LCSC PART NAME (none) -> C1779
- C68: renamed from C70; footprint (none) -> Capacitor_SMD:C_0805_2012Metric; LCSC PART NAME (none) -> C1779
- C69: renamed from C71; footprint (none) -> Capacitor_SMD:C_1206_3216Metric; LCSC PART NAME (none) -> C12891
- C70: renamed from C72; footprint (none) -> Capacitor_SMD:C_0805_2012Metric; LCSC PART NAME (none) -> C15850
- C71: renamed from C73; footprint (none) -> Capacitor_SMD:C_1206_3216Metric; LCSC PART NAME (none) -> C12891
- C72: renamed from C74; footprint (none) -> Capacitor_SMD:C_0805_2012Metric; LCSC PART NAME (none) -> C1779
- C73: renamed from C75; footprint (none) -> Capacitor_SMD:C_0805_2012Metric; LCSC PART NAME (none) -> C1779
- C74: renamed from C76; footprint (none) -> Capacitor_SMD:C_0805_2012Metric; LCSC PART NAME (none) -> C1779
- C75: renamed from C77; footprint (none) -> Capacitor_SMD:C_0805_2012Metric; LCSC PART NAME (none) -> C1779
- C76: renamed from C78; footprint (none) -> Capacitor_SMD:C_1206_3216Metric; LCSC PART NAME (none) -> C12891
- C77: renamed from C79; footprint (none) -> Capacitor_SMD:C_0805_2012Metric; LCSC PART NAME (none) -> C15850
- C78: renamed from C80; footprint (none) -> Capacitor_SMD:C_1206_3216Metric; LCSC PART NAME (none) -> C12891
- C79: renamed from C81; footprint (none) -> Capacitor_SMD:C_0805_2012Metric; LCSC PART NAME (none) -> C1779
- C80: renamed from C82; footprint (none) -> Capacitor_SMD:C_0805_2012Metric; LCSC PART NAME (none) -> C1779
- C81: renamed from C83; footprint (none) -> Capacitor_SMD:C_1206_3216Metric; LCSC PART NAME (none) -> C12891
- C82: renamed from C84; footprint (none) -> Capacitor_SMD:C_0805_2012Metric; LCSC PART NAME (none) -> C15850
- C83: renamed from C85; footprint (none) -> Capacitor_SMD:C_1206_3216Metric; LCSC PART NAME (none) -> C12891
- C84: renamed from C86; footprint (none) -> Capacitor_SMD:C_0805_2012Metric; LCSC PART NAME (none) -> C1779
- U5: LCSC PART NAME RK3566 -> (none)
Connections:
- net VDD_GPU_NPU: now also NT5.2
- net VDD_LOGIC: now also NT4.2
- new net FB1: NT4.1
- new net FB2: NT5.1
Other:
- sheet USB AVDD ports: added USB_OTG_DN, USB_OTG_DP; removed USB_DM, USB_DP
- moved on the sheet: C78, C79, C80, C83, C84

Commit message: Minor tweaks
Parts:
- renumbered NT4 to NT5, NT5 to NT6
Changed lines of the file:
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@@
 		(dnp no)
 		(fields_autoplaced yes)
-		(property "Reference" "NT5"
+		(property "Reference" "NT6"
 			(at 120.65 125.3955 0)
 			(effects
@@
 			(project ""
 				(path "/da62c771-e8c9-451f-8df1-ec995aadcb11/279fc251-45a8-41a3-8fcf-5855d7fe07da"
-					(reference "NT5")
+					(reference "NT6")
 					(unit 1)
 				)
@@
 		(dnp no)
 		(fields_autoplaced yes)
-		(property "Reference" "NT4"
+		(property "Reference" "NT5"
 			(at 120.65 83.4855 0)
 			(effects
@@
 			(project "srad-camera"
 				(path "/da62c771-e8c9-451f-8df1-ec995aadcb11/279fc251-45a8-41a3-8fcf-5855d7fe07da"
-					(reference "NT4")
+					(reference "NT5")
 					(unit 1)
 				)
