File: kicad/subsheets/imu.kicad_sch (KiCad schematic)
At the start: 5 parts

Commit message: Mark as R1.0
Parts:
- renumbered C50 to C51, C51 to C52, R27 to R29, R28 to R30
Other:
- company: (none) -> UVic Rocketry
Changed lines of the file:
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@@
 	(title_block
 		(title "Inertial Measurement Unit")
+		(date "2025-11-23")
+		(rev "1.0")
+		(company "UVic Rocketry")
+		(comment 1 "Author: Eric Handley")
 	)
 	(text "CS High for I2C"
@@
 		(on_board yes)
 		(dnp no)
-		(property "Reference" "R27"
+		(property "Reference" "R29"
 			(at 165.1 66.548 90)
 			(effects
@@
 			(project "srad-camera"
 				(path "/da62c771-e8c9-451f-8df1-ec995aadcb11/53c61148-5ca8-449f-9011-3672d8a04f56"
-					(reference "R27")
+					(reference "R29")
 					(unit 1)
 				)
@@
 		(on_board yes)
 		(dnp no)
-		(property "Reference" "C51"
+		(property "Reference" "C52"
 			(at 147.828 109.728 0)
 			(effects
@@
 			(project "srad-camera"
 				(path "/da62c771-e8c9-451f-8df1-ec995aadcb11/53c61148-5ca8-449f-9011-3672d8a04f56"
-					(reference "C51")
+					(reference "C52")
 					(unit 1)
 				)
@@
 		(on_board yes)
 		(dnp no)
-		(property "Reference" "#PWR038"
+		(property "Reference" "#PWR045"
 			(at 125.73 99.06 0)
 			(effects
@@
 			(project "srad-camera"
 				(path "/da62c771-e8c9-451f-8df1-ec995aadcb11/53c61148-5ca8-449f-9011-3672d8a04f56"
-					(reference "#PWR038")
+					(reference "#PWR045")
 					(unit 1)
 				)
@@
 		(on_board yes)
 		(dnp no)
-		(property "Reference" "#PWR039"
+		(property "Reference" "#PWR046"
 			(at 170.18 107.95 0)
 			(effects
@@
 			(project "srad-camera"
 				(path "/da62c771-e8c9-451f-8df1-ec995aadcb11/53c61148-5ca8-449f-9011-3672d8a04f56"
-					(reference "#PWR039")
+					(reference "#PWR046")
 					(unit 1)
 				)
@@
 		(on_board yes)
 		(dnp no)
-		(property "Reference" "C50"
+		(property "Reference" "C51"
 			(at 172.466 96.774 0)
 			(effects
@@
 			(project "srad-camera"
 				(path "/da62c771-e8c9-451f-8df1-ec995aadcb11/53c61148-5ca8-449f-9011-3672d8a04f56"
-					(reference "C50")
+					(reference "C51")
 					(unit 1)
 				)
@@
 		(on_board yes)
 		(dnp no)
-		(property "Reference" "#PWR040"
+		(property "Reference" "#PWR047"
 			(at 149.86 121.92 0)
 			(effects
@@
 			(project "srad-camera"
 				(path "/da62c771-e8c9-451f-8df1-ec995aadcb11/53c61148-5ca8-449f-9011-3672d8a04f56"
-					(reference "#PWR040")
+					(reference "#PWR047")
 					(unit 1)
 				)
@@
 		(on_board yes)
 		(dnp no)
-		(property "Reference" "R28"
+		(property "Reference" "R30"
 			(at 165.1 71.12 90)
 			(effects
@@
 			(project "srad-camera"
 				(path "/da62c771-e8c9-451f-8df1-ec995aadcb11/53c61148-5ca8-449f-9011-3672d8a04f56"
-					(reference "R28")
+					(reference "R30")
 					(unit 1)
 				)

Commit message: Annotations
Parts:
- renumbered C51 to C64, C52 to C65, R29 to R32, R30 to R33
Changed lines of the file:
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@@
 		(on_board yes)
 		(dnp no)
-		(property "Reference" "R29"
+		(property "Reference" "R32"
 			(at 165.1 66.548 90)
 			(effects
@@
 			(project "srad-camera"
 				(path "/da62c771-e8c9-451f-8df1-ec995aadcb11/53c61148-5ca8-449f-9011-3672d8a04f56"
-					(reference "R29")
+					(reference "R32")
 					(unit 1)
 				)
@@
 		(on_board yes)
 		(dnp no)
-		(property "Reference" "C52"
+		(property "Reference" "C65"
 			(at 147.828 109.728 0)
 			(effects
@@
 			(project "srad-camera"
 				(path "/da62c771-e8c9-451f-8df1-ec995aadcb11/53c61148-5ca8-449f-9011-3672d8a04f56"
-					(reference "C52")
+					(reference "C65")
 					(unit 1)
 				)
@@
 		(on_board yes)
 		(dnp no)
-		(property "Reference" "#PWR045"
+		(property "Reference" "#PWR055"
 			(at 125.73 99.06 0)
 			(effects
@@
 			(project "srad-camera"
 				(path "/da62c771-e8c9-451f-8df1-ec995aadcb11/53c61148-5ca8-449f-9011-3672d8a04f56"
-					(reference "#PWR045")
+					(reference "#PWR055")
 					(unit 1)
 				)
@@
 		(on_board yes)
 		(dnp no)
-		(property "Reference" "#PWR046"
+		(property "Reference" "#PWR056"
 			(at 170.18 107.95 0)
 			(effects
@@
 			(project "srad-camera"
 				(path "/da62c771-e8c9-451f-8df1-ec995aadcb11/53c61148-5ca8-449f-9011-3672d8a04f56"
-					(reference "#PWR046")
+					(reference "#PWR056")
 					(unit 1)
 				)
@@
 		(on_board yes)
 		(dnp no)
-		(property "Reference" "C51"
+		(property "Reference" "C64"
 			(at 172.466 96.774 0)
 			(effects
@@
 			(project "srad-camera"
 				(path "/da62c771-e8c9-451f-8df1-ec995aadcb11/53c61148-5ca8-449f-9011-3672d8a04f56"
-					(reference "C51")
+					(reference "C64")
 					(unit 1)
 				)
@@
 		(on_board yes)
 		(dnp no)
-		(property "Reference" "#PWR047"
+		(property "Reference" "#PWR057"
 			(at 149.86 121.92 0)
 			(effects
@@
 			(project "srad-camera"
 				(path "/da62c771-e8c9-451f-8df1-ec995aadcb11/53c61148-5ca8-449f-9011-3672d8a04f56"
-					(reference "#PWR047")
+					(reference "#PWR057")
 					(unit 1)
 				)
@@
 		(on_board yes)
 		(dnp no)
-		(property "Reference" "R30"
+		(property "Reference" "R33"
 			(at 165.1 71.12 90)
 			(effects
@@
 			(project "srad-camera"
 				(path "/da62c771-e8c9-451f-8df1-ec995aadcb11/53c61148-5ca8-449f-9011-3672d8a04f56"
-					(reference "R30")
+					(reference "R33")
 					(unit 1)
 				)

Commit message: Minor tweaks + annotations
Changed lines of the file:
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@@
 	(text "I2C 0x6A"
 		(exclude_from_sim no)
-		(at 130.048 86.868 0)
+		(at 129.54 89.154 0)
 		(effects
 			(font

Commit message: Start on PCB design
Parts:
- C62: renamed from C64; footprint (none) -> Capacitor_SMD:C_0402_1005Metric; LCSC PART NAME (none) -> C1525
- C63: renamed from C65; footprint (none) -> Capacitor_SMD:C_0402_1005Metric; LCSC PART NAME (none) -> C1525
- R33: renamed from R32; footprint (none) -> Resistor_SMD:R_0402_1005Metric; LCSC PART NAME (none) -> C25900
- R34: renamed from R33; footprint (none) -> Resistor_SMD:R_0402_1005Metric; LCSC PART NAME (none) -> C25900
Changed lines of the file:
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@@
 		(on_board yes)
 		(dnp no)
-		(property "Reference" "R32"
+		(property "Reference" "R33"
 			(at 165.1 66.548 90)
 			(effects
@@
 			)
 		)
-		(property "Footprint" ""
+		(property "Footprint" "Resistor_SMD:R_0402_1005Metric"
 			(at 158.75 69.85 0)
 			(effects
@@
 		)
 		(property "SUPPLEMENTARY FEATURES" ""
+			(at 158.75 69.85 90)
+			(effects
+				(font
+					(size 1.27 1.27)
+				)
+				(hide yes)
+			)
+		)
+		(property "LCSC PART NAME" "C25900"
 			(at 158.75 69.85 90)
 			(effects
@@
 			(project "srad-camera"
 				(path "/da62c771-e8c9-451f-8df1-ec995aadcb11/53c61148-5ca8-449f-9011-3672d8a04f56"
-					(reference "R32")
+					(reference "R33")
 					(unit 1)
 				)
@@
 		(on_board yes)
 		(dnp no)
-		(property "Reference" "C65"
+		(property "Reference" "C63"
 			(at 147.828 109.728 0)
 			(effects
@@
 			)
 		)
-		(property "Footprint" ""
+		(property "Footprint" "Capacitor_SMD:C_0402_1005Metric"
 			(at 149.86 110.49 0)
 			(effects
@@
 			)
 		)
-		(property "V" ""
+		(property "LCSC PART NAME" "C1525"
 			(at 149.86 110.49 0)
 			(effects
@@
 			(project "srad-camera"
 				(path "/da62c771-e8c9-451f-8df1-ec995aadcb11/53c61148-5ca8-449f-9011-3672d8a04f56"
-					(reference "C65")
+					(reference "C63")
 					(unit 1)
 				)
@@
 		(on_board yes)
 		(dnp no)
-		(property "Reference" "#PWR055"
+		(property "Reference" "#PWR054"
 			(at 125.73 99.06 0)
 			(effects
@@
 			(project "srad-camera"
 				(path "/da62c771-e8c9-451f-8df1-ec995aadcb11/53c61148-5ca8-449f-9011-3672d8a04f56"
-					(reference "#PWR055")
+					(reference "#PWR054")
 					(unit 1)
 				)
@@
 		(on_board yes)
 		(dnp no)
-		(property "Reference" "#PWR056"
+		(property "Reference" "#PWR055"
 			(at 170.18 107.95 0)
 			(effects
@@
 			(project "srad-camera"
 				(path "/da62c771-e8c9-451f-8df1-ec995aadcb11/53c61148-5ca8-449f-9011-3672d8a04f56"
-					(reference "#PWR056")
+					(reference "#PWR055")
 					(unit 1)
 				)
@@
 		(on_board yes)
 		(dnp no)
-		(property "Reference" "C64"
+		(property "Reference" "C62"
 			(at 172.466 96.774 0)
 			(effects
@@
 			)
 		)
-		(property "Footprint" ""
+		(property "Footprint" "Capacitor_SMD:C_0402_1005Metric"
 			(at 170.18 97.79 0)
 			(effects
@@
 			)
 		)
-		(property "V" ""
+		(property "LCSC PART NAME" "C1525"
 			(at 170.18 97.79 0)
 			(effects
@@
 			(project "srad-camera"
 				(path "/da62c771-e8c9-451f-8df1-ec995aadcb11/53c61148-5ca8-449f-9011-3672d8a04f56"
-					(reference "C64")
+					(reference "C62")
 					(unit 1)
 				)
@@
 		(on_board yes)
 		(dnp no)
-		(property "Reference" "#PWR057"
+		(property "Reference" "#PWR056"
 			(at 149.86 121.92 0)
 			(effects
@@
 			(project "srad-camera"
 				(path "/da62c771-e8c9-451f-8df1-ec995aadcb11/53c61148-5ca8-449f-9011-3672d8a04f56"
-					(reference "#PWR057")
+					(reference "#PWR056")
 					(unit 1)
 				)
@@
 		(on_board yes)
 		(dnp no)
-		(property "Reference" "R33"
+		(property "Reference" "R34"
 			(at 165.1 71.12 90)
 			(effects
@@
 			)
 		)
-		(property "Footprint" ""
+		(property "Footprint" "Resistor_SMD:R_0402_1005Metric"
 			(at 158.75 72.39 0)
 			(effects
@@
 		)
 		(property "SUPPLEMENTARY FEATURES" ""
+			(at 158.75 72.39 90)
+			(effects
+				(font
+					(size 1.27 1.27)
+				)
+				(hide yes)
+			)
+		)
+		(property "LCSC PART NAME" "C25900"
 			(at 158.75 72.39 90)
 			(effects
@@
 			(project "srad-camera"
 				(path "/da62c771-e8c9-451f-8df1-ec995aadcb11/53c61148-5ca8-449f-9011-3672d8a04f56"
-					(reference "R33")
+					(reference "R34")
 					(unit 1)
 				)
