File: kicad/subsheets/pmic.kicad_sch (KiCad schematic)
At the start: 66 parts, among them U3 RK809-5

Commit message: All major components placed on board
Parts:
- removed C42, C43: 22uF, Capacitor_SMD:C_1206_3216Metric, symbol Device:C_Small
- removed L7: 470nH / 4A, Inductor_SMD:L_0805_2012Metric, symbol Device:L_Small
Connections:
- net BUCK4_1V8: no longer names the net of U3.64 (FB4)
- net SW4: no longer names the net of U3.65 (SW4)
- no-connect marks 16 -> 18
Other:
- moved on the sheet: C17, C29, C30, C31, C35, C36, C37, C38, C47, C48, HSE1, L3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

Commit message: Allllmost everything placed
Parts:
- removed NT1: NetTie_2, symbol Device:NetTie_2
Connections:
- net VBUCK3 is gone; now on net BUCK3_1V35: C32.1, C33.1, C34.1, L4.2, R23.2, U3.26 (VBUCK3)
Changed lines of the file:
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@@
 	)
 	(junction
+		(at 193.04 63.5)
+		(diameter 0)
+		(color 0 0 0 0)
+	)
+	(junction
 		(at 120.65 99.06)
 		(diameter 0)
@@
 	)
 	(junction
-		(at 193.04 63.5)
-		(diameter 0)
-		(color 0 0 0 0)
-	)
-	(junction
 		(at 125.73 113.03)
 		(diameter 0)
@@
 	(wire
 		(pts
-			(xy 185.42 63.5) (xy 187.96 63.5)
+			(xy 185.42 63.5) (xy 193.04 63.5)
 		)
 		(stroke
@@
 					(unit 1)
 				)
-			)
-		)
-	)
-	(symbol
-		(lib_id "Device:NetTie_2")
-		(at 190.5 63.5 0)
-		(unit 1)
-		(exclude_from_sim no)
-		(in_bom no)
-		(on_board yes)
-		(dnp no)
-		(fields_autoplaced yes)
-		(property "Reference" "NT1"
-			(at 190.5 59.3555 0)
-			(effects
-				(font
-					(size 1.27 1.27)
-				)
-				(hide yes)
-			)
-		)
-		(property "Value" "NetTie_2"
-			(at 190.5 61.7798 0)
-			(effects
-				(font
-					(size 1.27 1.27)
-				)
-				(hide yes)
-			)
-		)
-		(property "Footprint" ""
-			(at 190.5 63.5 0)
-			(effects
-				(font
-					(size 1.27 1.27)
-				)
-				(hide yes)
-			)
-		)
-		(property "Datasheet" "~"
-			(at 190.5 63.5 0)
-			(effects
-				(font
-					(size 1.27 1.27)
-				)
-				(hide yes)
-			)
-		)
-		(property "Description" "Net tie, 2 pins"
-			(at 190.5 63.5 0)
-			(effects
-				(font
-					(size 1.27 1.27)
-				)
-				(hide yes)
-			)
-		)
-		(pin "2"
-		)
-		(pin "1"
-		)
-		(instances
-			(project "srad-camera"
-				(path "/da62c771-e8c9-451f-8df1-ec995aadcb11/6bb226bc-8621-46e9-a0f1-5501f65ad069"
-					(reference "NT1")
-					(unit 1)
-				)
