File: kicad/subsheets/stm32.kicad_sch (KiCad schematic)
At the start: 11 parts, among them U4 STM32U575RGT6

Commit message: Annotations
Parts:
- renumbered C42 to C55, C43 to C56, C44 to C57, C45 to C58, C46 to C59, C47 to C60, C48 to C61, C49 to C62, C50 to C63, R28 to R31
Changed lines of the file:
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@@
 		(on_board yes)
 		(dnp no)
-		(property "Reference" "#PWR043"
+		(property "Reference" "#PWR053"
 			(at 128.27 132.08 0)
 			(effects
@@
 			(project "srad-camera"
 				(path "/da62c771-e8c9-451f-8df1-ec995aadcb11/cf8a0c2d-fb2b-4eaa-949d-0ddbf6dd7299"
-					(reference "#PWR043")
+					(reference "#PWR053")
 					(unit 1)
 				)
@@
 		(on_board yes)
 		(dnp no)
-		(property "Reference" "C46"
+		(property "Reference" "C59"
 			(at 156.21 43.434 90)
 			(effects
@@
 			(project "srad-camera"
 				(path "/da62c771-e8c9-451f-8df1-ec995aadcb11/cf8a0c2d-fb2b-4eaa-949d-0ddbf6dd7299"
-					(reference "C46")
+					(reference "C59")
 					(unit 1)
 				)
@@
 		(on_board yes)
 		(dnp no)
-		(property "Reference" "C45"
+		(property "Reference" "C58"
 			(at 153.67 43.434 90)
 			(effects
@@
 			(project "srad-camera"
 				(path "/da62c771-e8c9-451f-8df1-ec995aadcb11/cf8a0c2d-fb2b-4eaa-949d-0ddbf6dd7299"
-					(reference "C45")
+					(reference "C58")
 					(unit 1)
 				)
@@
 		(on_board yes)
 		(dnp no)
-		(property "Reference" "C49"
+		(property "Reference" "C62"
 			(at 126.238 62.484 90)
 			(effects
@@
 			(project "srad-camera"
 				(path "/da62c771-e8c9-451f-8df1-ec995aadcb11/cf8a0c2d-fb2b-4eaa-949d-0ddbf6dd7299"
-					(reference "C49")
+					(reference "C62")
 					(unit 1)
 				)
@@
 		(on_board yes)
 		(dnp no)
-		(property "Reference" "C43"
+		(property "Reference" "C56"
 			(at 148.59 43.434 90)
 			(effects
@@
 			(project "srad-camera"
 				(path "/da62c771-e8c9-451f-8df1-ec995aadcb11/cf8a0c2d-fb2b-4eaa-949d-0ddbf6dd7299"
-					(reference "C43")
+					(reference "C56")
 					(unit 1)
 				)
@@
 		(on_board yes)
 		(dnp no)
-		(property "Reference" "#PWR042"
+		(property "Reference" "#PWR052"
 			(at 119.38 68.58 0)
 			(effects
@@
 			(project "srad-camera"
 				(path "/da62c771-e8c9-451f-8df1-ec995aadcb11/cf8a0c2d-fb2b-4eaa-949d-0ddbf6dd7299"
-					(reference "#PWR042")
+					(reference "#PWR052")
 					(unit 1)
 				)
@@
 		(on_board yes)
 		(dnp no)
-		(property "Reference" "C48"
+		(property "Reference" "C61"
 			(at 161.29 43.434 90)
 			(effects
@@
 			(project "srad-camera"
 				(path "/da62c771-e8c9-451f-8df1-ec995aadcb11/cf8a0c2d-fb2b-4eaa-949d-0ddbf6dd7299"
-					(reference "C48")
+					(reference "C61")
 					(unit 1)
 				)
@@
 		(on_board yes)
 		(dnp no)
-		(property "Reference" "C44"
+		(property "Reference" "C57"
 			(at 151.13 43.434 90)
 			(effects
@@
 			(project "srad-camera"
 				(path "/da62c771-e8c9-451f-8df1-ec995aadcb11/cf8a0c2d-fb2b-4eaa-949d-0ddbf6dd7299"
-					(reference "C44")
+					(reference "C57")
 					(unit 1)
 				)
@@
 		(on_board yes)
 		(dnp no)
-		(property "Reference" "C42"
+		(property "Reference" "C55"
 			(at 143.51 43.434 90)
 			(effects
@@
 			(project "srad-camera"
 				(path "/da62c771-e8c9-451f-8df1-ec995aadcb11/cf8a0c2d-fb2b-4eaa-949d-0ddbf6dd7299"
-					(reference "C42")
+					(reference "C55")
 					(unit 1)
 				)
@@
 		(on_board yes)
 		(dnp no)
-		(property "Reference" "C50"
+		(property "Reference" "C63"
 			(at 130.81 121.158 90)
 			(effects
@@
 			(project "srad-camera"
 				(path "/da62c771-e8c9-451f-8df1-ec995aadcb11/cf8a0c2d-fb2b-4eaa-949d-0ddbf6dd7299"
-					(reference "C50")
+					(reference "C63")
 					(unit 1)
 				)
@@
 		(on_board yes)
 		(dnp no)
-		(property "Reference" "#PWR044"
+		(property "Reference" "#PWR054"
 			(at 153.67 154.94 0)
 			(effects
@@
 			(project "srad-camera"
 				(path "/da62c771-e8c9-451f-8df1-ec995aadcb11/cf8a0c2d-fb2b-4eaa-949d-0ddbf6dd7299"
-					(reference "#PWR044")
+					(reference "#PWR054")
 					(unit 1)
 				)
@@
 		(on_board yes)
 		(dnp no)
-		(property "Reference" "#PWR041"
+		(property "Reference" "#PWR051"
 			(at 166.37 53.34 0)
 			(effects
@@
 			(project ""
 				(path "/da62c771-e8c9-451f-8df1-ec995aadcb11/cf8a0c2d-fb2b-4eaa-949d-0ddbf6dd7299"
-					(reference "#PWR041")
+					(reference "#PWR051")
 					(unit 1)
 				)
@@
 		(on_board yes)
 		(dnp no)
-		(property "Reference" "R28"
+		(property "Reference" "R31"
 			(at 127 73.406 90)
 			(effects
@@
 			(project "srad-camera"
 				(path "/da62c771-e8c9-451f-8df1-ec995aadcb11/cf8a0c2d-fb2b-4eaa-949d-0ddbf6dd7299"
-					(reference "R28")
+					(reference "R31")
 					(unit 1)
 				)
@@
 		(on_board yes)
 		(dnp no)
-		(property "Reference" "C47"
+		(property "Reference" "C60"
 			(at 158.75 43.434 90)
 			(effects
@@
 			(project "srad-camera"
 				(path "/da62c771-e8c9-451f-8df1-ec995aadcb11/cf8a0c2d-fb2b-4eaa-949d-0ddbf6dd7299"
-					(reference "C47")
+					(reference "C60")
 					(unit 1)
 				)

Commit message: Start on PCB design
Parts:
- C53: renamed from C55; footprint (none) -> Capacitor_SMD:C_0805_2012Metric; LCSC PART NAME (none) -> C15850
- C54: renamed from C56; footprint (none) -> Capacitor_SMD:C_0402_1005Metric; LCSC PART NAME (none) -> C1525
- C55: renamed from C57; footprint (none) -> Capacitor_SMD:C_0402_1005Metric; LCSC PART NAME (none) -> C1525
- C56: renamed from C58; footprint (none) -> Capacitor_SMD:C_0402_1005Metric; LCSC PART NAME (none) -> C1525
- C57: renamed from C59; footprint (none) -> Capacitor_SMD:C_0402_1005Metric; LCSC PART NAME (none) -> C1525
- C58: renamed from C60; footprint (none) -> Capacitor_SMD:C_0402_1005Metric; LCSC PART NAME (none) -> C1525
- C59: renamed from C61; footprint (none) -> Capacitor_SMD:C_0402_1005Metric; LCSC PART NAME (none) -> C1525
- C60: renamed from C62; footprint (none) -> Capacitor_SMD:C_0402_1005Metric; LCSC PART NAME (none) -> C1525
- C61: renamed from C63; value 4.7uF 20% -> 4.7uF; footprint (none) -> Capacitor_SMD:C_0805_2012Metric; LCSC PART NAME (none) -> C1779
- R32: renamed from R31; value 1k -> 4.7k; footprint (none) -> Resistor_SMD:R_0402_1005Metric; LCSC PART NAME (none) -> C25900
Changed lines of the file:
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@@
 		(on_board yes)
 		(dnp no)
-		(property "Reference" "#PWR053"
+		(property "Reference" "#PWR052"
 			(at 128.27 132.08 0)
 			(effects
@@
 			(project "srad-camera"
 				(path "/da62c771-e8c9-451f-8df1-ec995aadcb11/cf8a0c2d-fb2b-4eaa-949d-0ddbf6dd7299"
-					(reference "#PWR053")
+					(reference "#PWR052")
 					(unit 1)
 				)
@@
 		(on_board yes)
 		(dnp no)
-		(property "Reference" "C59"
+		(property "Reference" "C57"
 			(at 156.21 43.434 90)
 			(effects
@@
 			)
 		)
-		(property "Footprint" ""
+		(property "Footprint" "Capacitor_SMD:C_0402_1005Metric"
 			(at 156.21 48.26 0)
 			(effects
@@
 			)
 		)
-		(property "V" ""
+		(property "LCSC PART NAME" "C1525"
 			(at 156.21 48.26 90)
 			(effects
@@
 			(project "srad-camera"
 				(path "/da62c771-e8c9-451f-8df1-ec995aadcb11/cf8a0c2d-fb2b-4eaa-949d-0ddbf6dd7299"
-					(reference "C59")
+					(reference "C57")
 					(unit 1)
 				)
@@
 		(on_board yes)
 		(dnp no)
-		(property "Reference" "C58"
+		(property "Reference" "C56"
 			(at 153.67 43.434 90)
 			(effects
@@
 			)
 		)
-		(property "Footprint" ""
+		(property "Footprint" "Capacitor_SMD:C_0402_1005Metric"
 			(at 153.67 48.26 0)
 			(effects
@@
 			)
 		)
-		(property "V" ""
+		(property "LCSC PART NAME" "C1525"
 			(at 153.67 48.26 90)
 			(effects
@@
 			(project "srad-camera"
 				(path "/da62c771-e8c9-451f-8df1-ec995aadcb11/cf8a0c2d-fb2b-4eaa-949d-0ddbf6dd7299"
-					(reference "C58")
+					(reference "C56")
 					(unit 1)
 				)
@@
 		(on_board yes)
 		(dnp no)
-		(property "Reference" "C62"
+		(property "Reference" "C60"
 			(at 126.238 62.484 90)
 			(effects
@@
 			)
 		)
-		(property "Footprint" ""
+		(property "Footprint" "Capacitor_SMD:C_0402_1005Metric"
 			(at 123.19 60.96 0)
 			(effects
@@
 			)
 		)
-		(property "V" ""
+		(property "LCSC PART NAME" "C1525"
 			(at 123.19 60.96 90)
 			(effects
@@
 			(project "srad-camera"
 				(path "/da62c771-e8c9-451f-8df1-ec995aadcb11/cf8a0c2d-fb2b-4eaa-949d-0ddbf6dd7299"
-					(reference "C62")
+					(reference "C60")
 					(unit 1)
 				)
@@
 		(on_board yes)
 		(dnp no)
-		(property "Reference" "C56"
+		(property "Reference" "C54"
 			(at 148.59 43.434 90)
 			(effects
@@
 			)
 		)
-		(property "Footprint" ""
+		(property "Footprint" "Capacitor_SMD:C_0402_1005Metric"
 			(at 148.59 48.26 0)
 			(effects
@@
 			)
 		)
-		(property "V" ""
+		(property "LCSC PART NAME" "C1525"
 			(at 148.59 48.26 90)
 			(effects
@@
 			(project "srad-camera"
 				(path "/da62c771-e8c9-451f-8df1-ec995aadcb11/cf8a0c2d-fb2b-4eaa-949d-0ddbf6dd7299"
-					(reference "C56")
+					(reference "C54")
 					(unit 1)
 				)
@@
 		(on_board yes)
 		(dnp no)
-		(property "Reference" "#PWR052"
+		(property "Reference" "#PWR051"
 			(at 119.38 68.58 0)
 			(effects
@@
 			(project "srad-camera"
 				(path "/da62c771-e8c9-451f-8df1-ec995aadcb11/cf8a0c2d-fb2b-4eaa-949d-0ddbf6dd7299"
-					(reference "#PWR052")
+					(reference "#PWR051")
 					(unit 1)
 				)
@@
 		(on_board yes)
 		(dnp no)
-		(property "Reference" "C61"
+		(property "Reference" "C59"
 			(at 161.29 43.434 90)
 			(effects
@@
 			)
 		)
-		(property "Footprint" ""
+		(property "Footprint" "Capacitor_SMD:C_0402_1005Metric"
 			(at 161.29 48.26 0)
 			(effects
@@
 			)
 		)
-		(property "V" ""
+		(property "LCSC PART NAME" "C1525"
 			(at 161.29 48.26 90)
 			(effects
@@
 			(project "srad-camera"
 				(path "/da62c771-e8c9-451f-8df1-ec995aadcb11/cf8a0c2d-fb2b-4eaa-949d-0ddbf6dd7299"
-					(reference "C61")
+					(reference "C59")
 					(unit 1)
 				)
@@
 		(on_board yes)
 		(dnp no)
-		(property "Reference" "C57"
+		(property "Reference" "C55"
 			(at 151.13 43.434 90)
 			(effects
@@
 			)
 		)
-		(property "Footprint" ""
+		(property "Footprint" "Capacitor_SMD:C_0402_1005Metric"
 			(at 151.13 48.26 0)
 			(effects
@@
 			)
 		)
-		(property "V" ""
+		(property "LCSC PART NAME" "C1525"
 			(at 151.13 48.26 90)
 			(effects
@@
 			(project "srad-camera"
 				(path "/da62c771-e8c9-451f-8df1-ec995aadcb11/cf8a0c2d-fb2b-4eaa-949d-0ddbf6dd7299"
-					(reference "C57")
+					(reference "C55")
 					(unit 1)
 				)
@@
 		(on_board yes)
 		(dnp no)
-		(property "Reference" "C55"
+		(property "Reference" "C53"
 			(at 143.51 43.434 90)
 			(effects
@@
 			)
 		)
-		(property "Footprint" ""
+		(property "Footprint" "Capacitor_SMD:C_0805_2012Metric"
 			(at 143.51 48.26 0)
 			(effects
@@
 		)
 		(property "SUPPLEMENTARY FEATURES" ""
+			(at 143.51 48.26 90)
+			(effects
+				(font
+					(size 1.27 1.27)
+				)
+				(hide yes)
+			)
+		)
+		(property "LCSC PART NAME" "C15850"
 			(at 143.51 48.26 90)
 			(effects
@@
 			(project "srad-camera"
 				(path "/da62c771-e8c9-451f-8df1-ec995aadcb11/cf8a0c2d-fb2b-4eaa-949d-0ddbf6dd7299"
-					(reference "C55")
+					(reference "C53")
 					(unit 1)
 				)
@@
 		(on_board yes)
 		(dnp no)
-		(property "Reference" "C63"
+		(property "Reference" "C61"
 			(at 130.81 121.158 90)
 			(effects
@@
 			)
 		)
-		(property "Value" "4.7uF 20%"
+		(property "Value" "4.7uF"
 			(at 130.81 122.936 90)
 			(effects
@@
 			)
 		)
-		(property "Footprint" ""
+		(property "Footprint" "Capacitor_SMD:C_0805_2012Metric"
 			(at 132.08 124.46 0)
 			(effects
@@
 		)
 		(property "SUPPLEMENTARY FEATURES" ""
+			(at 132.08 124.46 90)
+			(effects
+				(font
+					(size 1.27 1.27)
+				)
+				(hide yes)
+			)
+		)
+		(property "LCSC PART NAME" "C1779"
 			(at 132.08 124.46 90)
 			(effects
@@
 			(project "srad-camera"
 				(path "/da62c771-e8c9-451f-8df1-ec995aadcb11/cf8a0c2d-fb2b-4eaa-949d-0ddbf6dd7299"
-					(reference "C63")
+					(reference "C61")
 					(unit 1)
 				)
@@
 		(on_board yes)
 		(dnp no)
-		(property "Reference" "#FLG03"
+		(property "Reference" "#FLG05"
 			(at 135.89 48.895 0)
 			(effects
@@
 			(project "srad-camera"
 				(path "/da62c771-e8c9-451f-8df1-ec995aadcb11/cf8a0c2d-fb2b-4eaa-949d-0ddbf6dd7299"
-					(reference "#FLG03")
+					(reference "#FLG05")
 					(unit 1)
 				)
@@
 		(on_board yes)
 		(dnp no)
-		(property "Reference" "#PWR054"
+		(property "Reference" "#PWR053"
 			(at 153.67 154.94 0)
 			(effects
@@
 			(project "srad-camera"
 				(path "/da62c771-e8c9-451f-8df1-ec995aadcb11/cf8a0c2d-fb2b-4eaa-949d-0ddbf6dd7299"
-					(reference "#PWR054")
+					(reference "#PWR053")
 					(unit 1)
 				)
@@
 		(on_board yes)
 		(dnp no)
-		(property "Reference" "#PWR051"
+		(property "Reference" "#PWR050"
 			(at 166.37 53.34 0)
 			(effects
@@
 			(project ""
 				(path "/da62c771-e8c9-451f-8df1-ec995aadcb11/cf8a0c2d-fb2b-4eaa-949d-0ddbf6dd7299"
-					(reference "#PWR051")
+					(reference "#PWR050")
 					(unit 1)
 				)
@@
 		(on_board yes)
 		(dnp no)
-		(property "Reference" "R31"
+		(property "Reference" "R32"
 			(at 127 73.406 90)
 			(effects
@@
 			)
 		)
-		(property "Value" "1k"
+		(property "Value" "4.7k"
 			(at 127 75.184 90)
 			(effects
@@
 			)
 		)
-		(property "Footprint" ""
+		(property "Footprint" "Resistor_SMD:R_0402_1005Metric"
 			(at 127 71.12 0)
 			(effects
@@
 		)
 		(property "SUPPLEMENTARY FEATURES" ""
+			(at 127 71.12 90)
+			(effects
+				(font
+					(size 1.27 1.27)
+				)
+				(hide yes)
+			)
+		)
+		(property "LCSC PART NAME" "C25900"
 			(at 127 71.12 90)
 			(effects
@@
 			(project "srad-camera"
 				(path "/da62c771-e8c9-451f-8df1-ec995aadcb11/cf8a0c2d-fb2b-4eaa-949d-0ddbf6dd7299"
-					(reference "R31")
+					(reference "R32")
 					(unit 1)
 				)
@@
 		(on_board yes)
 		(dnp no)
-		(property "Reference" "C60"
+		(property "Reference" "C58"
 			(at 158.75 43.434 90)
 			(effects
@@
 			)
 		)
-		(property "Footprint" ""
+		(property "Footprint" "Capacitor_SMD:C_0402_1005Metric"
 			(at 158.75 48.26 0)
 			(effects
@@
 			)
 		)
-		(property "V" ""
+		(property "LCSC PART NAME" "C1525"
 			(at 158.75 48.26 90)
 			(effects
@@
 			(project "srad-camera"
 				(path "/da62c771-e8c9-451f-8df1-ec995aadcb11/cf8a0c2d-fb2b-4eaa-949d-0ddbf6dd7299"
-					(reference "C60")
+					(reference "C58")
 					(unit 1)
 				)
