File: kicad/subsheets/ddr3l.kicad_sch (KiCad schematic)
At the start: 34 parts, among them U6 MT41K256M16TW-107:P

Commit message: Minor tweaks + annotations
Connections:
- net +0.675V renamed V_{REFCA}
Other:
- note added: "+0.675V"
- note added: "+1.35V"
Changed lines of the file:
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@@
 		)
 	)
+	(text "+1.35V"
+		(exclude_from_sim no)
+		(at 199.644 123.952 0)
+		(effects
+			(font
+				(size 0.8 0.8)
+				(italic yes)
+			)
+		)
+	)
+	(text "+0.675V"
+		(exclude_from_sim no)
+		(at 213.868 123.952 0)
+		(effects
+			(font
+				(size 0.8 0.8)
+				(italic yes)
+			)
+		)
+	)
 	(junction
 		(at 194.31 92.71)
@@
 		)
 	)
-	(label "+0.675V"
-		(at 210.82 124.46 0)
-		(effects
-			(font
-				(size 0.8 0.8)
-				(italic yes)
-			)
-			(justify left bottom)
-		)
-	)
 	(label "DQS_P0"
 		(at 137.16 99.06 180)
@@
 		)
 	)
-	(label "+1.35V"
-		(at 203.2 124.46 180)
-		(effects
-			(font
-				(size 0.8 0.8)
-				(italic yes)
-			)
-			(justify right bottom)
-		)
-	)

Commit message: Start on PCB design
Parts:
- added R55: 120R, Resistor_SMD:R_0402_1005Metric, symbol Device:R_Small
- C137: renamed from C139; footprint (none) -> Capacitor_SMD:C_1206_3216Metric; LCSC PART NAME (none) -> C12891
- C138: renamed from C140; footprint (none) -> Capacitor_SMD:C_0805_2012Metric; LCSC PART NAME (none) -> C1779
- C139: renamed from C141; footprint (none) -> Capacitor_SMD:C_0805_2012Metric; LCSC PART NAME (none) -> C1779
- C140: renamed from C142; footprint (none) -> Capacitor_SMD:C_0402_1005Metric; LCSC PART NAME (none) -> C1525
- C141: renamed from C143; footprint (none) -> Capacitor_SMD:C_0402_1005Metric; LCSC PART NAME (none) -> C1525
- C142: renamed from C144; footprint (none) -> Capacitor_SMD:C_0402_1005Metric; LCSC PART NAME (none) -> C1525
- C143: renamed from C145; footprint (none) -> Capacitor_SMD:C_0402_1005Metric; LCSC PART NAME (none) -> C1525
- C144: renamed from C146; footprint (none) -> Capacitor_SMD:C_0402_1005Metric; LCSC PART NAME (none) -> C1525
- C145: renamed from C147; footprint (none) -> Capacitor_SMD:C_0402_1005Metric; LCSC PART NAME (none) -> C1525
- C146: renamed from C148; footprint (none) -> Capacitor_SMD:C_0402_1005Metric; LCSC PART NAME (none) -> C1525
- C147: renamed from C149; footprint (none) -> Capacitor_SMD:C_0402_1005Metric; LCSC PART NAME (none) -> C1525
- C148: renamed from C150; footprint (none) -> Capacitor_SMD:C_0402_1005Metric; LCSC PART NAME (none) -> C1525
- C149: renamed from C151; footprint (none) -> Capacitor_SMD:C_1206_3216Metric; LCSC PART NAME (none) -> C12891
- C150: renamed from C152; footprint (none) -> Capacitor_SMD:C_0805_2012Metric; LCSC PART NAME (none) -> C1779
- C151: renamed from C153; footprint (none) -> Capacitor_SMD:C_0805_2012Metric; LCSC PART NAME (none) -> C1779
- C152: renamed from C154; footprint (none) -> Capacitor_SMD:C_0402_1005Metric; LCSC PART NAME (none) -> C1525
- C153: renamed from C155; footprint (none) -> Capacitor_SMD:C_0402_1005Metric; LCSC PART NAME (none) -> C1525
- C154: renamed from C156; footprint (none) -> Capacitor_SMD:C_0402_1005Metric; LCSC PART NAME (none) -> C1525
- C155: renamed from C157; footprint (none) -> Capacitor_SMD:C_0402_1005Metric; LCSC PART NAME (none) -> C1525
- C156: renamed from C158; footprint (none) -> Capacitor_SMD:C_0402_1005Metric; LCSC PART NAME (none) -> C1525
- C157: renamed from C159; footprint (none) -> Capacitor_SMD:C_0402_1005Metric; LCSC PART NAME (none) -> C1525
- C158: renamed from C160; footprint (none) -> Capacitor_SMD:C_0402_1005Metric; LCSC PART NAME (none) -> C1525
- C159: renamed from C161; footprint (none) -> Capacitor_SMD:C_0402_1005Metric; LCSC PART NAME (none) -> C1525
- C160: renamed from C162; footprint (none) -> Capacitor_SMD:C_0402_1005Metric; LCSC PART NAME (none) -> C1525
- C161: renamed from C163; footprint (none) -> Capacitor_SMD:C_0402_1005Metric; LCSC PART NAME (none) -> C1525
- C162: renamed from C164; footprint (none) -> Capacitor_SMD:C_0402_1005Metric; LCSC PART NAME (none) -> C1525
- C163: renamed from C165; footprint (none) -> Capacitor_SMD:C_0402_1005Metric; LCSC PART NAME (none) -> C1525
- C164: renamed from C166; footprint (none) -> Capacitor_SMD:C_0402_1005Metric; LCSC PART NAME (none) -> C1523
- R50: renamed from R49; footprint (none) -> Resistor_SMD:R_0603_1608Metric; LCSC PART NAME (none) -> C25804
- R51: renamed from R50; footprint (none) -> Resistor_SMD:R_0603_1608Metric; LCSC PART NAME (none) -> C25804
- R52: renamed from R51; value 240 -> 220R; footprint (none) -> Resistor_SMD:R_0603_1608Metric; LCSC PART NAME (none) -> C22962
- R53: renamed from R52; value 240 -> 220R; footprint (none) -> Resistor_SMD:R_0603_1608Metric; LCSC PART NAME (none) -> C22962
- R54: renamed from R53; value 240 -> 120R; footprint (none) -> Resistor_SMD:R_0402_1005Metric; LCSC PART NAME (none) -> C25079
Connections:
- net GND: now also R55.1; no longer R54.1
- new net: R54.1, R55.2

Commit message: Remove power/decoupling for unused power domains
Parts:
- renumbered C137 to C123, C138 to C124, C139 to C125, C140 to C126, C141 to C127, C142 to C128, C143 to C129, C144 to C130, C145 to C131, C146 to C132, C147 to C133, C148 to C134, C149 to C135, C150 to C136, C151 to C137, C152 to C138, C153 to C139, C154 to C140, C155 to C141, C156 to C142, C157 to C143, C158 to C144, C159 to C145, C160 to C146, C161 to C147, C162 to C148, C163 to C149, C164 to C150, R50 to R47, R51 to R48, R52 to R49, R53 to R50, R54 to R51, R55 to R52
