File: kicad/srad-camera.kicad_pcb (KiCad board)
At the start: 2 copper layers, 0 parts

Commit message: Start on PCB design
Parts:
- added C1: 1uF, Capacitor_SMD:C_0603_1608Metric, F.Cu at (88.5, 62.9)
- added C10: 10uF, Capacitor_SMD:C_0805_2012Metric, B.Cu at (254.7, 55.4)
- added C100: 100nF, Capacitor_SMD:C_0402_1005Metric, F.Cu at (86.5, 23.4)
- added C101: 1uF, Capacitor_SMD:C_0603_1608Metric, F.Cu at (80.1, 23.7)
- added C102: 22pF, Capacitor_SMD:C_0402_1005Metric, F.Cu at (86.5, 25.4)
- added C103: 100nF, Capacitor_SMD:C_0402_1005Metric, F.Cu at (86.5, 27.4)
- added C104: 22pF, Capacitor_SMD:C_0402_1005Metric, F.Cu at (86.5, 29.3)
- added C105: 1uF, Capacitor_SMD:C_0603_1608Metric, F.Cu at (80.1, 26.2)
- added C106: 100nF, Capacitor_SMD:C_0402_1005Metric, F.Cu at (86.5, 31.3)
- added C107: 1uF, Capacitor_SMD:C_0603_1608Metric, F.Cu at (80.1, 28.7)
- added C108: 100nF, Capacitor_SMD:C_0402_1005Metric, F.Cu at (89.3, 23.4)
- added C109: 1uF, Capacitor_SMD:C_0603_1608Metric, F.Cu at (80.1, 31.2)
- added C11: 10uF, Capacitor_SMD:C_0805_2012Metric, B.Cu at (255.2, 61.5)
- added C110: 100nF, Capacitor_SMD:C_0402_1005Metric, F.Cu at (89.3, 25.4)
- added C111: 1uF, Capacitor_SMD:C_0603_1608Metric, F.Cu at (80.1, 33.7)
- added C112: 100nF, Capacitor_SMD:C_0402_1005Metric, F.Cu at (89.3, 27.4)
- added C113: 100nF, Capacitor_SMD:C_0402_1005Metric, F.Cu at (89.3, 29.3)
- added C114: 100nF, Capacitor_SMD:C_0402_1005Metric, F.Cu at (89.3, 31.3)
- added C115: 100nF, Capacitor_SMD:C_0402_1005Metric, F.Cu at (82.5, 38.9)
- added C116: 100nF, Capacitor_SMD:C_0402_1005Metric, F.Cu at (82.5, 40.9)
- added C117: 100nF, Capacitor_SMD:C_0402_1005Metric, F.Cu at (82.5, 42.9)
- added C118: 100nF, Capacitor_SMD:C_0402_1005Metric, F.Cu at (85.3, 38.9)
- added C119: 100nF, Capacitor_SMD:C_0402_1005Metric, F.Cu at (85.3, 40.9)
- added C12: 1uF, Capacitor_SMD:C_0603_1608Metric, B.Cu at (256.5, 55.2)
- added C120: 100nF, Capacitor_SMD:C_0402_1005Metric, F.Cu at (85.3, 42.9)
- added C121: 100nF, Capacitor_SMD:C_0402_1005Metric, F.Cu at (88.2, 38.9)
- added C122: 100nF, Capacitor_SMD:C_0402_1005Metric, F.Cu at (88.2, 40.9)
- added C123: 100nF, Capacitor_SMD:C_0402_1005Metric, F.Cu at (88.2, 42.9)
- added C124: 100nF, Capacitor_SMD:C_0402_1005Metric, F.Cu at (94.2, 23.4)
- added C125: 100nF, Capacitor_SMD:C_0402_1005Metric, F.Cu at (94.2, 25.4)
- added C126: 100nF, Capacitor_SMD:C_0402_1005Metric, F.Cu at (94.2, 27.4)
- added C127: 100nF, Capacitor_SMD:C_0402_1005Metric, F.Cu at (94.2, 29.3)
- added C128: 1uF, Capacitor_SMD:C_0603_1608Metric, F.Cu at (39.9, 81.3)
- added C129: 100nF, Capacitor_SMD:C_0402_1005Metric, F.Cu at (36.5, 81.0)
- added C13: 1uF, Capacitor_SMD:C_0603_1608Metric, B.Cu at (252.7, 55.0)
- added C130: 100nF, Capacitor_SMD:C_0402_1005Metric, F.Cu at (36.5, 83.0)
- added C131: 100nF, Capacitor_SMD:C_0402_1005Metric, F.Cu at (36.5, 85.0)
- added C132: 100nF, Capacitor_SMD:C_0402_1005Metric, F.Cu at (36.5, 86.9)
- added C133: 100nF, Capacitor_SMD:C_0402_1005Metric, F.Cu at (36.5, 88.9)
- added C134: 100nF, Capacitor_SMD:C_0402_1005Metric, F.Cu at (36.5, 90.9)
- added C135: 100nF, Capacitor_SMD:C_0402_1005Metric, F.Cu at (36.5, 92.8)
- added C136: 100nF, Capacitor_SMD:C_0402_1005Metric, F.Cu at (36.5, 94.8)
- added C137: 22uF, Capacitor_SMD:C_1206_3216Metric, F.Cu at (49.9, 73.3)
- added C138: 4.7uF, Capacitor_SMD:C_0805_2012Metric, F.Cu at (60.4, 56.1)
- added C139: 4.7uF, Capacitor_SMD:C_0805_2012Metric, F.Cu at (60.4, 59.1)
- added C14: 1uF, Capacitor_SMD:C_0603_1608Metric, B.Cu at (257.7, 60.5)
- added C140: 100nF, Capacitor_SMD:C_0402_1005Metric, F.Cu at (59.6, 67.6)
- added C141: 100nF, Capacitor_SMD:C_0402_1005Metric, F.Cu at (59.6, 69.6)
- added C142: 100nF, Capacitor_SMD:C_0402_1005Metric, F.Cu at (59.6, 71.5)
- added C143: 100nF, Capacitor_SMD:C_0402_1005Metric, F.Cu at (59.6, 73.5)
- added C144: 100nF, Capacitor_SMD:C_0402_1005Metric, F.Cu at (59.6, 75.5)
- added C145: 100nF, Capacitor_SMD:C_0402_1005Metric, F.Cu at (59.6, 77.5)
- added C146: 100nF, Capacitor_SMD:C_0402_1005Metric, F.Cu at (62.4, 67.6)
- added C147: 100nF, Capacitor_SMD:C_0402_1005Metric, F.Cu at (62.4, 69.6)
- added C148: 100nF, Capacitor_SMD:C_0402_1005Metric, F.Cu at (62.4, 71.5)
- added C149: 22uF, Capacitor_SMD:C_1206_3216Metric, F.Cu at (49.9, 76.7)
- added C15: 1uF, Capacitor_SMD:C_0603_1608Metric, B.Cu at (252.9, 60.9)
- added C150: 4.7uF, Capacitor_SMD:C_0805_2012Metric, F.Cu at (60.4, 62.1)
- added C151: 4.7uF, Capacitor_SMD:C_0805_2012Metric, F.Cu at (60.4, 65.1)
- added C152: 100nF, Capacitor_SMD:C_0402_1005Metric, F.Cu at (62.4, 73.5)
- added C153: 100nF, Capacitor_SMD:C_0402_1005Metric, F.Cu at (62.4, 75.5)
- added C154: 100nF, Capacitor_SMD:C_0402_1005Metric, F.Cu at (62.4, 77.5)
- added C155: 100nF, Capacitor_SMD:C_0402_1005Metric, F.Cu at (65.3, 67.6)
- added C156: 100nF, Capacitor_SMD:C_0402_1005Metric, F.Cu at (65.3, 69.6)
- added C157: 100nF, Capacitor_SMD:C_0402_1005Metric, F.Cu at (65.3, 71.5)
- added C158: 100nF, Capacitor_SMD:C_0402_1005Metric, F.Cu at (65.3, 73.5)
- added C159: 100nF, Capacitor_SMD:C_0402_1005Metric, F.Cu at (65.3, 75.5)
- added C16: 10uF, Capacitor_SMD:C_0805_2012Metric, B.Cu at (251.1, 60.6)
- added C160: 100nF, Capacitor_SMD:C_0402_1005Metric, F.Cu at (65.3, 77.5)
- added C161: 100nF, Capacitor_SMD:C_0402_1005Metric, F.Cu at (68.2, 67.6)
- added C162: 100nF, Capacitor_SMD:C_0402_1005Metric, F.Cu at (68.2, 69.6)
- added C163: 100nF, Capacitor_SMD:C_0402_1005Metric, F.Cu at (68.2, 71.5)
- added C164: 1nF, Capacitor_SMD:C_0402_1005Metric, F.Cu at (68.2, 73.5)
- added C165: 100nF, Capacitor_SMD:C_0402_1005Metric, F.Cu at (31.3, 71.6)
- added C166: 1uF, Capacitor_SMD:C_0603_1608Metric, F.Cu at (27.4, 74.9)
- added C167: 10uF, Capacitor_SMD:C_0805_2012Metric, F.Cu at (27.6, 72.1)
- added C17: 100nF, Capacitor_SMD:C_0402_1005Metric, F.Cu at (262.4, 56.2)
- added C18: 1uF, Capacitor_SMD:C_0603_1608Metric, B.Cu at (259.5, 58.7)
- added C19: 1uF, Capacitor_SMD:C_0603_1608Metric, F.Cu at (259.7, 60.1)
- added C2: 22uF, Capacitor_SMD:C_1206_3216Metric, F.Cu at (143.2, 25.6)
- added C20: 1uF, Capacitor_SMD:C_0603_1608Metric, F.Cu at (260.4, 61.7)
- added C21: 1uF, Capacitor_SMD:C_0603_1608Metric, B.Cu at (250.6, 54.7)
- added C22: 1uF, Capacitor_SMD:C_0603_1608Metric, B.Cu at (250.7, 51.6)
- added C23: 1uF, Capacitor_SMD:C_0603_1608Metric, F.Cu at (249.5, 53.4)
- added C24: 1uF, Capacitor_SMD:C_0603_1608Metric, F.Cu at (259.4, 55.0)
- added C25: 1uF, Capacitor_SMD:C_0603_1608Metric, F.Cu at (258.3, 53.5)
- added C26: 1uF, Capacitor_SMD:C_0603_1608Metric, F.Cu at (256.0, 52.0)
- added C27: 1uF, Capacitor_SMD:C_0603_1608Metric, F.Cu at (253.5, 63.9)
- added C28: 1uF, Capacitor_SMD:C_0603_1608Metric, F.Cu at (252.0, 64.2)
- added C29: 10uF, Capacitor_SMD:C_0805_2012Metric, B.Cu at (260.3, 56.2)
- added C3: 22uF, Capacitor_SMD:C_1206_3216Metric, F.Cu at (150.6, 25.5)
- added C30: 22uF, Capacitor_SMD:C_1206_3216Metric, B.Cu at (262.5, 55.7)
- added C31: 22uF, Capacitor_SMD:C_1206_3216Metric, B.Cu at (264.8, 55.6)
- added C32: 10uF, Capacitor_SMD:C_0805_2012Metric, B.Cu at (255.4, 51.6)
- added C33: 22uF, Capacitor_SMD:C_1206_3216Metric, B.Cu at (253.2, 50.9)
- added C34: 10uF, Capacitor_SMD:C_0805_2012Metric, B.Cu at (249.2, 46.9)
- added C35: 100nF, Capacitor_SMD:C_0402_1005Metric, F.Cu at (263.6, 58.6)
- added C36: 10uF, Capacitor_SMD:C_0805_2012Metric, B.Cu at (262.4, 59.8)
- added C37: 22uF, Capacitor_SMD:C_1206_3216Metric, B.Cu at (264.6, 60.3)
- added C38: 22uF, Capacitor_SMD:C_1206_3216Metric, F.Cu at (271.2, 58.3)
- added C39: 10uF, Capacitor_SMD:C_0805_2012Metric, F.Cu at (259.8, 77.7)
- added C4: 22uF, Capacitor_SMD:C_1206_3216Metric, F.Cu at (143.1, 30.2)
- added C40: 22uF, Capacitor_SMD:C_1206_3216Metric, F.Cu at (260.4, 71.8)
- added C41: 10uF, Capacitor_SMD:C_0805_2012Metric, F.Cu at (262.1, 74.9)
- added C42: 22uF, Capacitor_SMD:C_1206_3216Metric, F.Cu at (256.7, 69.1)
- added C43: 10uF, Capacitor_SMD:C_0805_2012Metric, F.Cu at (254.5, 70.2)
- added C43: 22uF, Capacitor_SMD:C_1206_3216Metric, F.Cu at (252.2, 70.5)
- added C44: 1uF, Capacitor_SMD:C_0603_1608Metric, F.Cu at (246.4, 56.5)
- added C45: 1uF, Capacitor_SMD:C_0603_1608Metric, F.Cu at (248.7, 54.9)
- added C46: 1uF, Capacitor_SMD:C_0603_1608Metric, F.Cu at (248.7, 56.4)
- added C47: 22pf, Capacitor_SMD:C_0402_1005Metric, F.Cu at (246.4, 61.4)
- added C48: 22pf, Capacitor_SMD:C_0402_1005Metric, F.Cu at (246.4, 63.5)
- added C49: 1uF, Capacitor_SMD:C_0603_1608Metric, F.Cu at (248.7, 58.0)
- added C5: 22uF, Capacitor_SMD:C_1206_3216Metric, F.Cu at (150.6, 30.2)
- added C50: 1uF, Capacitor_SMD:C_0603_1608Metric, B.Cu at (248.8, 59.0)
- added C51: 1uF, Capacitor_SMD:C_0603_1608Metric, B.Cu at (251.1, 58.2)
- added C52: 1uF, Capacitor_SMD:C_0603_1608Metric, F.Cu at (248.0, 59.6)
- added C53: 10uF, Capacitor_SMD:C_0805_2012Metric, F.Cu at (73.8, 95.8)
- added C54: 100nF, Capacitor_SMD:C_0402_1005Metric, F.Cu at (87.5, 80.9)
- added C55: 100nF, Capacitor_SMD:C_0402_1005Metric, F.Cu at (87.5, 82.8)
- added C56: 100nF, Capacitor_SMD:C_0402_1005Metric, F.Cu at (87.5, 84.8)
- added C57: 100nF, Capacitor_SMD:C_0402_1005Metric, F.Cu at (87.5, 86.8)
- added C58: 100nF, Capacitor_SMD:C_0402_1005Metric, F.Cu at (87.5, 88.8)
- added C59: 100nF, Capacitor_SMD:C_0402_1005Metric, F.Cu at (87.5, 90.7)
- added C6: 10uF, Capacitor_SMD:C_0805_2012Metric, F.Cu at (199.3, 115.6)
- added C60: 100nF, Capacitor_SMD:C_0402_1005Metric, F.Cu at (87.5, 92.7)
- added C61: 4.7uF, Capacitor_SMD:C_0805_2012Metric, F.Cu at (197.1, 59.1)
- added C62: 100nF, Capacitor_SMD:C_0402_1005Metric, F.Cu at (92.4, 84.9)
- added C63: 100nF, Capacitor_SMD:C_0402_1005Metric, F.Cu at (189.5, 60.7)
- added C64: 22uF, Capacitor_SMD:C_1206_3216Metric, F.Cu at (55.5, 24.1)
- added C65: 22uF, Capacitor_SMD:C_1206_3216Metric, F.Cu at (55.5, 27.4)
- added C66: 22uF, Capacitor_SMD:C_1206_3216Metric, F.Cu at (55.5, 30.8)
- added C67: 4.7uF, Capacitor_SMD:C_0805_2012Metric, F.Cu at (74.1, 47.5)
- added C68: 4.7uF, Capacitor_SMD:C_0805_2012Metric, F.Cu at (60.6, 43.0)
- added C69: 22uF, Capacitor_SMD:C_1206_3216Metric, F.Cu at (55.5, 34.1)
- added C7: 100nF, Capacitor_SMD:C_0402_1005Metric, F.Cu at (184.9, 106.5)
- added C70: 10uF, Capacitor_SMD:C_0805_2012Metric, F.Cu at (60.6, 46.0)
- added C71: 22uF, Capacitor_SMD:C_1206_3216Metric, F.Cu at (55.5, 37.5)
- added C72: 4.7uF, Capacitor_SMD:C_0805_2012Metric, F.Cu at (60.6, 49.0)
- added C73: 4.7uF, Capacitor_SMD:C_0805_2012Metric, F.Cu at (65.0, 40.0)
- added C74: 4.7uF, Capacitor_SMD:C_0805_2012Metric, F.Cu at (65.0, 43.0)
- added C75: 4.7uF, Capacitor_SMD:C_0805_2012Metric, F.Cu at (65.0, 46.0)
- added C76: 22uF, Capacitor_SMD:C_1206_3216Metric, F.Cu at (55.5, 40.9)
- added C77: 10uF, Capacitor_SMD:C_0805_2012Metric, F.Cu at (65.0, 49.0)
- added C78: 22uF, Capacitor_SMD:C_1206_3216Metric, F.Cu at (55.5, 44.2)
- added C79: 4.7uF, Capacitor_SMD:C_0805_2012Metric, F.Cu at (69.5, 40.0)
- added C8: 10uF, Capacitor_SMD:C_0805_2012Metric, B.Cu at (258.3, 56.0)
- added C80: 4.7uF, Capacitor_SMD:C_0805_2012Metric, F.Cu at (69.5, 43.0)
- added C81: 22uF, Capacitor_SMD:C_1206_3216Metric, F.Cu at (55.5, 47.5)
- added C82: 10uF, Capacitor_SMD:C_0805_2012Metric, F.Cu at (69.5, 46.0)
- added C83: 22uF, Capacitor_SMD:C_1206_3216Metric, F.Cu at (55.5, 50.9)
- added C84: 4.7uF, Capacitor_SMD:C_0805_2012Metric, F.Cu at (69.5, 49.0)
- added C85: 100nF, Capacitor_SMD:C_0402_1005Metric, F.Cu at (92.4, 90.9)
- added C86: 100nF, Capacitor_SMD:C_0402_1005Metric, F.Cu at (92.4, 92.8)
- added C87: 100nF, Capacitor_SMD:C_0402_1005Metric, F.Cu at (92.4, 94.8)
- added C88: 100nF, Capacitor_SMD:C_0402_1005Metric, F.Cu at (92.4, 96.8)
- added C89: 1nF, Capacitor_SMD:C_0402_1005Metric, F.Cu at (92.4, 98.7)
- added C9: 10uF, Capacitor_SMD:C_0805_2012Metric, B.Cu at (256.3, 58.7)
- added C90: 100nF, Capacitor_SMD:C_0402_1005Metric, F.Cu at (97.5, 40.9)
- added C91: 100nF, Capacitor_SMD:C_0402_1005Metric, F.Cu at (97.5, 42.9)
- added C92: 100nF, Capacitor_SMD:C_0402_1005Metric, F.Cu at (97.5, 44.8)
- added C93: 4.7uF, Capacitor_SMD:C_0805_2012Metric, F.Cu at (93.9, 39.4)
- added C94: 4.7uF, Capacitor_SMD:C_0805_2012Metric, F.Cu at (93.9, 42.4)
- added C95: 100nF, Capacitor_SMD:C_0402_1005Metric, F.Cu at (97.5, 46.8)
- added C96: 100nF, Capacitor_SMD:C_0402_1005Metric, F.Cu at (97.5, 48.8)
- added C97: 100nF, Capacitor_SMD:C_0402_1005Metric, F.Cu at (97.5, 50.8)
- added C98: 4.7uF, Capacitor_SMD:C_0805_2012Metric, F.Cu at (93.9, 45.5)
- added C99: 4.7uF, Capacitor_SMD:C_0805_2012Metric, F.Cu at (93.9, 48.5)
- added D1: SMAJ5.0A, Diode_SMD:D_SMA, F.Cu at (183.3, 113.3)
- added D10: TVS Vr3.3 Vb4, Diode_SMD:D_SOD-123F, F.Cu at (53.4, 139.6)
- added D2: TVS Vr3.3 Vb4, Diode_SMD:D_SOD-123F, F.Cu at (195.4, 97.6)
- added D3: TVS Vr3.3 Vb4, Diode_SMD:D_SOD-123F, F.Cu at (195.4, 102.1)
- added D4: TVS Vr3.3 Vb4, Diode_SMD:D_SOD-123F, F.Cu at (53.4, 119.5)
- added D5: TVS Vr3.3 Vb4, Diode_SMD:D_SOD-123F, F.Cu at (53.4, 122.8)
- added D6: TVS Vr3.3 Vb4, Diode_SMD:D_SOD-123F, F.Cu at (53.4, 126.2)
- added D7: TVS Vr3.3 Vb4, Diode_SMD:D_SOD-123F, F.Cu at (53.4, 129.5)
- added D8: TVS Vr3.3 Vb4, Diode_SMD:D_SOD-123F, F.Cu at (53.4, 132.9)
- added D9: TVS Vr3.3 Vb4, Diode_SMD:D_SOD-123F, F.Cu at (53.4, 136.2)
- added FB1: 120R, Resistor_SMD:R_0201_0603Metric, F.Cu at (91.7, 62.5)
- added FB2: 120R, Resistor_SMD:R_0201_0603Metric, F.Cu at (196.2, 119.5)
- added FB3: 120R, Resistor_SMD:R_0201_0603Metric, F.Cu at (198.3, 106.8)
- added FPC1: 0.5K-AX-22PWB, srad-camera-footprints:FPC-SMD_22P-P0.50_HDGC_0.5K-AX-22PWB, F.Cu at (146.5, 122.5)
- added HSE1: 32.768kHz, Crystal:Crystal_SMD_3215-2Pin_3.2x1.5mm, F.Cu at (248.1, 62.4)
- added HSE2: 24MHz, Crystal:Crystal_SMD_2016-4Pin_2.0x1.6mm, F.Cu at (87.1, 34.1)
- added IMU1: LSM6DSRTR, Package_LGA:LGA-14_3x2.5mm_P0.5mm_LayoutBorder3x4y, F.Cu at (191.5, 60.7)
- added J1: DEBUG, Connector_PinHeader_1.27mm:PinHeader_2x05_P1.27mm_Vertical_SMD, F.Cu at (211.1, 74.0)
- added JST1: XHP-3, Connector_JST:JST_XH_B3B-XH-A_1x03_P2.50mm_Vertical, F.Cu at (139.1, 25.4)
- added JST2: XHP-2, Connector_JST:JST_XH_B2B-XH-A_1x02_P2.50mm_Vertical, F.Cu at (207.5, 56.5)
- added L1: 1uH, Inductor_SMD:L_0805_2012Metric, F.Cu at (148.4, 26.2)
- added L2: 680nH, Inductor_SMD:L_0603_1608Metric, F.Cu at (148.4, 29.7)
- added L3: 470nH / 4A, Inductor_SMD:L_0805_2012Metric, F.Cu at (259.6, 57.2)
- added L4: 470nH / 4A, Inductor_SMD:L_0805_2012Metric, F.Cu at (254.4, 51.7)
- added L5: 470nH / 4A, Inductor_SMD:L_0805_2012Metric, F.Cu at (262.3, 59.1)
- added L6: 470nH / 4A, Inductor_SMD:L_0805_2012Metric, F.Cu at (250.4, 64.1)
- added L7: 470nH / 4A, Inductor_SMD:L_0805_2012Metric, F.Cu at (256.1, 74.9)
- added LED1: 150141GS63140, LED_SMD:LED_0805_2012Metric, F.Cu at (260.8, 52.5)
- added R1: 10k, Resistor_SMD:R_0402_1005Metric, F.Cu at (73.1, 62.7)
- added R10: 22k, Resistor_SMD:R_0402_1005Metric, F.Cu at (147.4, 23.9)
- added R11: 200k, Resistor_SMD:R_0402_1005Metric, F.Cu at (146.2, 30.8)
- added R12: 200k, Resistor_SMD:R_0402_1005Metric, F.Cu at (145.3, 31.9)
- added R13: 200k, Resistor_SMD:R_0402_1005Metric, F.Cu at (147.2, 31.9)
- added R14: 5.1k, Resistor_SMD:R_0402_1005Metric, F.Cu at (197.0, 97.6)
- added R15: 5.1k, Resistor_SMD:R_0402_1005Metric, F.Cu at (197.0, 101.8)
- added R16: 22R, Resistor_SMD:R_0402_1005Metric, F.Cu at (193.2, 100.4)
- added R17: 22R, Resistor_SMD:R_0402_1005Metric, F.Cu at (193.3, 99.4)
- added R18: 1M, Resistor_SMD:R_0402_1005Metric, F.Cu at (200.3, 106.8)
- added R19: 10k, Resistor_SMD:R_0402_1005Metric, F.Cu at (180.0, 98.8)
- added R2: 10k, Resistor_SMD:R_0402_1005Metric, F.Cu at (73.1, 64.7)
- added R20: 10k, Resistor_SMD:R_0402_1005Metric, F.Cu at (184.0, 98.8)
- added R21: 100R, Resistor_SMD:R_0402_1005Metric, F.Cu at (261.9, 55.3)
- added R22: 120k, Resistor_SMD:R_0603_1608Metric, F.Cu at (251.1, 51.2)
- added R23: 82k, Resistor_SMD:R_0603_1608Metric, F.Cu at (252.6, 51.2)
- added R24: 100R, Resistor_SMD:R_0402_1005Metric, F.Cu at (260.5, 58.7)
- added R25: 10k, Resistor_SMD:R_0402_1005Metric, F.Cu at (253.5, 66.8)
- added R26: 4.7k, Resistor_SMD:R_0402_1005Metric, F.Cu at (260.4, 63.0)
- added R27: 4.7k, Resistor_SMD:R_0402_1005Metric, F.Cu at (260.4, 64.0)
- added R28: 10k, Resistor_SMD:R_0402_1005Metric, F.Cu at (258.2, 63.0)
- added R29: 10k, Resistor_SMD:R_0402_1005Metric, F.Cu at (257.5, 63.7)
- added R3: 10k, Resistor_SMD:R_0402_1005Metric, F.Cu at (73.1, 66.7)
- added R30: 10k, Resistor_SMD:R_0402_1005Metric, F.Cu at (261.9, 63.5)
- added R31: 220R, Resistor_SMD:R_0603_1608Metric, F.Cu at (258.3, 51.6)
- added R32: 4.7k, Resistor_SMD:R_0402_1005Metric, F.Cu at (77.5, 95.3)
- added R33: 4.7k, Resistor_SMD:R_0402_1005Metric, F.Cu at (193.5, 61.4)
- added R34: 4.7k, Resistor_SMD:R_0402_1005Metric, F.Cu at (191.5, 58.4)
- added R35: 10k, Resistor_SMD:R_0402_1005Metric, F.Cu at (95.2, 90.9)
- added R36: 120R, Resistor_SMD:R_0402_1005Metric, F.Cu at (97.5, 38.9)
- added R37: 22R, Resistor_SMD:R_0402_1005Metric, F.Cu at (83.6, 23.4)
- added R38: 0R, Resistor_SMD:R_0402_1005Metric, F.Cu at (83.6, 25.4)
- added R39: 1M, Resistor_SMD:R_0402_1005Metric, F.Cu at (83.6, 27.4)
- added R4: 22R, Resistor_SMD:R_0402_1005Metric, F.Cu at (205.8, 76.5)
- added R40: 0R, Resistor_SMD:R_0402_1005Metric, F.Cu at (83.6, 29.4)
- added R41: 100R, Resistor_SMD:R_0402_1005Metric, F.Cu at (83.6, 31.4)
- added R42: 0R, Resistor_SMD:R_0402_1005Metric, F.Cu at (79.6, 38.9)
- added R43: 1R, Resistor_SMD:R_0402_1005Metric, F.Cu at (79.6, 40.9)
- added R44: 1R, Resistor_SMD:R_0402_1005Metric, F.Cu at (79.6, 42.9)
- added R45: 1R, Resistor_SMD:R_0402_1005Metric, F.Cu at (79.6, 44.9)
- added R46: 1R, Resistor_SMD:R_0402_1005Metric, F.Cu at (79.6, 46.9)
- added R47: 0R, Resistor_SMD:R_0402_1005Metric, F.Cu at (79.6, 48.9)
- added R48: 22R, Resistor_SMD:R_0402_1005Metric, F.Cu at (97.1, 23.4)
- added R49: 1R, Resistor_SMD:R_0402_1005Metric, F.Cu at (39.4, 83.5)
- added R5: 22R, Resistor_SMD:R_0402_1005Metric, F.Cu at (205.8, 75.2)
- added R50: 10k, Resistor_SMD:R_0603_1608Metric, F.Cu at (64.6, 55.8)
- added R51: 10k, Resistor_SMD:R_0603_1608Metric, F.Cu at (64.6, 58.3)
- added R52: 220R, Resistor_SMD:R_0603_1608Metric, F.Cu at (64.6, 60.9)
- added R53: 220R, Resistor_SMD:R_0603_1608Metric, F.Cu at (64.6, 63.4)
- added R54: 120R, Resistor_SMD:R_0402_1005Metric, F.Cu at (54.2, 72.6)
- added R55: 120R, Resistor_SMD:R_0402_1005Metric, F.Cu at (54.2, 74.6)
- added R56: 22R, Resistor_SMD:R_0402_1005Metric, F.Cu at (68.2, 131.9)
- added R57: 22R, Resistor_SMD:R_0402_1005Metric, F.Cu at (68.2, 129.9)
- added R58: 22R, Resistor_SMD:R_0402_1005Metric, F.Cu at (68.2, 127.9)
- added R59: 22R, Resistor_SMD:R_0402_1005Metric, F.Cu at (68.2, 125.9)
- added R6: 4.7k, Resistor_SMD:R_0402_1005Metric, F.Cu at (73.1, 72.6)
- added R60: 22R, Resistor_SMD:R_0402_1005Metric, F.Cu at (68.2, 123.9)
- added R61: 22R, Resistor_SMD:R_0402_1005Metric, F.Cu at (68.2, 121.9)
- added R7: 4.7k, Resistor_SMD:R_0402_1005Metric, F.Cu at (73.1, 74.6)
- added R8: 200k, Resistor_SMD:R_0402_1005Metric, F.Cu at (146.3, 25.2)
- added R9: 22k, Resistor_SMD:R_0402_1005Metric, F.Cu at (145.5, 23.9)
- added SD1: MOLEX 472192001, Connector_Card:microSD_HC_Molex_47219-2001, F.Cu at (73.3, 150.0)
- added U1: AP61300Z6, Package_TO_SOT_SMD:SOT-563, F.Cu at (146.2, 26.6)
- added U2: AP61300Z6, Package_TO_SOT_SMD:SOT-563, F.Cu at (146.2, 29.4)
- added U3: RK809-5, Package_DFN_QFN:ArtInChip_QFN-68-1EP_7x7mm_P0.35mm_EP5.49x5.49mm, F.Cu at (254.0, 58.3)
- added U4: STM32U575RGT6, Package_QFP:LQFP-64_10x10mm_P0.5mm, F.Cu at (199.8, 67.5)
- added U5: RK3566, srad-camera-footprints:BGA-565_L15.5-W14.4-P0.40_RK3566_1, F.Cu at (146.0, 102.2)
- added U6: MT41K256M16TW-107:P, Package_BGA:Micron_FBGA-96_8x14mm_Layout9x16_P0.8mm, F.Cu at (127.1, 102.9)
- added USB1: 12402012E212A, srad-camera-footprints:USB-SMD_TYPE-C16PIN-1, F.Cu at (200.8, 99.9)
Routing:
- net GND: track 0.00 -> 34.6 mm, vias 0 -> 30
- net VCC_3V3_SYS: track 0.00 -> 24.8 mm, vias 0 -> 8
- net BUCK5_2V2: track 0.00 -> 19.8 mm, vias 0 -> 2
- net /Power Supply/VIN_5V: track 0.00 -> 17.1 mm
- net /STM32U575RGT6/SWDIO: track 0.00 -> 16.6 mm
- net VCCIO_3V3_IMU: track 0.00 -> 15.3 mm, vias 0 -> 1
- net (no net): track 0.00 -> 12.6 mm
- net /STM32U575RGT6/SWO: track 0.00 -> 11.3 mm
- net /LSM6DSRTR/SDA: track 0.00 -> 11.3 mm, vias 0 -> 2
- net /STM32U575RGT6/VDD_3V3: track 0.00 -> 11.1 mm, vias 0 -> 7
- net /STM32U575RGT6/SWCLK: track 0.00 -> 10.6 mm
- net /RK3566 SoC/VDD_LOGIC: track 0.00 -> 9.83 mm, vias 0 -> 1
- net VCC_0V9_CPU: track 0.00 -> 9.55 mm
- net /RK3566 SoC/VDD_GPU_NPU: track 0.00 -> 9.54 mm, vias 0 -> 1
- net FB1: track 0.00 -> 8.60 mm
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- added copper zone on In2.Cu, net /STM32U575RGT6/VDD_3V3
- added copper zone on In1.Cu, net GND
- added copper zone on In2.Cu, net VCC_3V3_SYS
Other:
- copper layers 2 -> 4
- board text added: "SCREWS!!!!!"
