File: kicad/srad-camera.kicad_pcb (KiCad board)
At the start: 4 copper layers, 50 x 50 mm, 247 parts, among them J1 DEBUG, SW1 PWR, SW2 USER, SW3 BOOT0, U1 AP61300Z6, U2 AP61300Z6, U3 RK809-5, U4 STM32U575RGT6, U5 RK3566, U6 MT41K256M16TW-107:P

Commit message: Restructure repo
Parts:
- moved R34 1.32 mm to (94.3, 43.0), turned to 0 degrees
- moved R33 1.26 mm to (92.8, 44.1), turned to 180 degrees
- moved C62 0.72 mm to (92.7, 42.1), turned to 180 degrees
Connections:
- H2 pad 1: GND -> unconnected-(H2-MP-Pad1)
- H3 pad 1: GND -> unconnected-(H3-MP-Pad1)
- H4 pad 1: GND -> unconnected-(H4-MP-Pad1)
Routing:
- net VCC_DDR: track 173.6 -> 121.7 mm
- net VCCIO_3V3_IMU: track 73.9 -> 59.8 mm
- net GND: track 351.3 -> 345.8 mm, vias 254 -> 252
- net /LSM6DSRTR/INT1: track 16.1 -> 12.7 mm
- net /LSM6DSRTR/SDA: track 14.9 -> 12.5 mm
- net /STM32U575RGT6/NRST: track 21.3 -> 19.3 mm
- net /LSM6DSRTR/SCL: track 15.5 -> 17.3 mm
- added copper zone on In2.Cu, net VCCIO_3V3_IMU
- removed copper zone on F.Cu, net GND
