File: kicad/subsheets/rk-domains/mipi-csi-dsi-hdmi.kicad_sch (KiCad schematic)
At the start: 11 parts, among them U5 RK3566

Commit message: Mark as R1.0
Parts:
- renumbered C145 to C117, C146 to C118, C148 to C119, C149 to C120, C150 to C121, C114 to C122, C115 to C123, C151 to C124, C152 to C125, R51 to R45
Other:
- company: (none) -> UVic Rocketry
Changed lines of the file:
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@@
 	(title_block
 		(title "MIPI CSI/DSI, HDMI")
+		(date "2025-11-23")
+		(rev "1.0")
+		(company "UVic Rocketry")
+		(comment 1 "Author: Eric Handley")
 	)
 	(junction
@@
 		(on_board yes)
 		(dnp no)
-		(property "Reference" "C150"
+		(property "Reference" "C121"
 			(at 221.742 88.3855 0)
 			(effects
@@
 			(project "srad-camera"
 				(path "/da62c771-e8c9-451f-8df1-ec995aadcb11/279fc251-45a8-41a3-8fcf-5855d7fe07da/ebdbfe46-9733-485c-9ca3-58f0449d57c1"
-					(reference "C150")
+					(reference "C121")
 					(unit 1)
 				)
@@
 		(dnp no)
 		(fields_autoplaced yes)
-		(property "Reference" "#PWR060"
+		(property "Reference" "#PWR087"
 			(at 88.9 107.95 0)
 			(effects
@@
 			(project "srad-camera"
 				(path "/da62c771-e8c9-451f-8df1-ec995aadcb11/279fc251-45a8-41a3-8fcf-5855d7fe07da/ebdbfe46-9733-485c-9ca3-58f0449d57c1"
-					(reference "#PWR060")
+					(reference "#PWR087")
 					(unit 1)
 				)
@@
 		(on_board yes)
 		(dnp no)
-		(property "Reference" "#PWR087"
+		(property "Reference" "#PWR089"
 			(at 96.52 137.16 0)
 			(effects
@@
 			(project "srad-camera"
 				(path "/da62c771-e8c9-451f-8df1-ec995aadcb11/279fc251-45a8-41a3-8fcf-5855d7fe07da/ebdbfe46-9733-485c-9ca3-58f0449d57c1"
-					(reference "#PWR087")
+					(reference "#PWR089")
 					(unit 1)
 				)
@@
 		(dnp no)
 		(fields_autoplaced yes)
-		(property "Reference" "#PWR082"
+		(property "Reference" "#PWR086"
 			(at 91.44 92.71 0)
 			(effects
@@
 			(project "srad-camera"
 				(path "/da62c771-e8c9-451f-8df1-ec995aadcb11/279fc251-45a8-41a3-8fcf-5855d7fe07da/ebdbfe46-9733-485c-9ca3-58f0449d57c1"
-					(reference "#PWR082")
+					(reference "#PWR086")
 					(unit 1)
 				)
@@
 		(on_board yes)
 		(dnp no)
-		(property "Reference" "#PWR086"
+		(property "Reference" "#PWR084"
 			(at 224.79 77.47 0)
 			(effects
@@
 			(project "srad-camera"
 				(path "/da62c771-e8c9-451f-8df1-ec995aadcb11/279fc251-45a8-41a3-8fcf-5855d7fe07da/ebdbfe46-9733-485c-9ca3-58f0449d57c1"
-					(reference "#PWR086")
+					(reference "#PWR084")
 					(unit 1)
 				)
@@
 		(on_board yes)
 		(dnp no)
-		(property "Reference" "C152"
+		(property "Reference" "C125"
 			(at 94.488 126.238 0)
 			(effects
@@
 			(project "srad-camera"
 				(path "/da62c771-e8c9-451f-8df1-ec995aadcb11/279fc251-45a8-41a3-8fcf-5855d7fe07da/ebdbfe46-9733-485c-9ca3-58f0449d57c1"
-					(reference "C152")
+					(reference "C125")
 					(unit 1)
 				)
@@
 		(dnp no)
 		(fields_autoplaced yes)
-		(property "Reference" "#FLG01"
+		(property "Reference" "#FLG07"
 			(at 222.25 57.785 0)
 			(effects
@@
 			(project "srad-camera"
 				(path "/da62c771-e8c9-451f-8df1-ec995aadcb11/279fc251-45a8-41a3-8fcf-5855d7fe07da/ebdbfe46-9733-485c-9ca3-58f0449d57c1"
-					(reference "#FLG01")
+					(reference "#FLG07")
 					(unit 1)
 				)
@@
 		(on_board yes)
 		(dnp no)
-		(property "Reference" "C146"
+		(property "Reference" "C118"
 			(at 213.868 66.548 0)
 			(effects
@@
 			(project "srad-camera"
 				(path "/da62c771-e8c9-451f-8df1-ec995aadcb11/279fc251-45a8-41a3-8fcf-5855d7fe07da/ebdbfe46-9733-485c-9ca3-58f0449d57c1"
-					(reference "C146")
+					(reference "C118")
 					(unit 1)
 				)
@@
 		(dnp no)
 		(fields_autoplaced yes)
-		(property "Reference" "#PWR080"
+		(property "Reference" "#PWR082"
 			(at 148.59 46.99 0)
 			(effects
@@
 			(project "srad-camera"
 				(path "/da62c771-e8c9-451f-8df1-ec995aadcb11/279fc251-45a8-41a3-8fcf-5855d7fe07da/ebdbfe46-9733-485c-9ca3-58f0449d57c1"
-					(reference "#PWR080")
+					(reference "#PWR082")
 					(unit 1)
 				)
@@
 		(on_board yes)
 		(dnp no)
-		(property "Reference" "C151"
+		(property "Reference" "C124"
 			(at 210.312 124.968 0)
 			(effects
@@
 			(project "srad-camera"
 				(path "/da62c771-e8c9-451f-8df1-ec995aadcb11/279fc251-45a8-41a3-8fcf-5855d7fe07da/ebdbfe46-9733-485c-9ca3-58f0449d57c1"
-					(reference "C151")
+					(reference "C124")
 					(unit 1)
 				)
@@
 		(on_board yes)
 		(dnp no)
-		(property "Reference" "#PWR085"
+		(property "Reference" "#PWR088"
 			(at 208.28 135.89 0)
 			(effects
@@
 			(project "srad-camera"
 				(path "/da62c771-e8c9-451f-8df1-ec995aadcb11/279fc251-45a8-41a3-8fcf-5855d7fe07da/ebdbfe46-9733-485c-9ca3-58f0449d57c1"
-					(reference "#PWR085")
+					(reference "#PWR088")
 					(unit 1)
 				)
@@
 		(on_board yes)
 		(dnp no)
-		(property "Reference" "#PWR084"
+		(property "Reference" "#PWR085"
 			(at 219.71 91.44 0)
 			(effects
@@
 			(project "srad-camera"
 				(path "/da62c771-e8c9-451f-8df1-ec995aadcb11/279fc251-45a8-41a3-8fcf-5855d7fe07da/ebdbfe46-9733-485c-9ca3-58f0449d57c1"
-					(reference "#PWR084")
+					(reference "#PWR085")
 					(unit 1)
 				)
@@
 		(dnp no)
 		(fields_autoplaced yes)
-		(property "Reference" "C115"
+		(property "Reference" "C123"
 			(at 94.488 95.758 0)
 			(effects
@@
 			(project "srad-camera"
 				(path "/da62c771-e8c9-451f-8df1-ec995aadcb11/279fc251-45a8-41a3-8fcf-5855d7fe07da/ebdbfe46-9733-485c-9ca3-58f0449d57c1"
-					(reference "C115")
+					(reference "C123")
 					(unit 1)
 				)
@@
 		(dnp no)
 		(fields_autoplaced yes)
-		(property "Reference" "C114"
+		(property "Reference" "C122"
 			(at 87.122 95.758 0)
 			(effects
@@
 			(project "srad-camera"
 				(path "/da62c771-e8c9-451f-8df1-ec995aadcb11/279fc251-45a8-41a3-8fcf-5855d7fe07da/ebdbfe46-9733-485c-9ca3-58f0449d57c1"
-					(reference "C114")
+					(reference "C122")
 					(unit 1)
 				)
@@
 		(on_board yes)
 		(dnp no)
-		(property "Reference" "C148"
+		(property "Reference" "C119"
 			(at 221.742 66.5545 0)
 			(effects
@@
 			(project "srad-camera"
 				(path "/da62c771-e8c9-451f-8df1-ec995aadcb11/279fc251-45a8-41a3-8fcf-5855d7fe07da/ebdbfe46-9733-485c-9ca3-58f0449d57c1"
-					(reference "C148")
+					(reference "C119")
 					(unit 1)
 				)
@@
 		(on_board yes)
 		(dnp no)
-		(property "Reference" "R51"
+		(property "Reference" "R45"
 			(at 152.4 35.4767 90)
 			(effects
@@
 			(project "srad-camera"
 				(path "/da62c771-e8c9-451f-8df1-ec995aadcb11/279fc251-45a8-41a3-8fcf-5855d7fe07da/ebdbfe46-9733-485c-9ca3-58f0449d57c1"
-					(reference "R51")
+					(reference "R45")
 					(unit 1)
 				)
@@
 		(dnp no)
 		(fields_autoplaced yes)
-		(property "Reference" "C145"
+		(property "Reference" "C117"
 			(at 146.266 35.6114 0)
 			(effects
@@
 			(project "srad-camera"
 				(path "/da62c771-e8c9-451f-8df1-ec995aadcb11/279fc251-45a8-41a3-8fcf-5855d7fe07da/ebdbfe46-9733-485c-9ca3-58f0449d57c1"
-					(reference "C145")
+					(reference "C117")
 					(unit 1)
 				)
@@
 		(on_board yes)
 		(dnp no)
-		(property "Reference" "C149"
+		(property "Reference" "C120"
 			(at 213.868 88.392 0)
 			(effects
@@
 			(project "srad-camera"
 				(path "/da62c771-e8c9-451f-8df1-ec995aadcb11/279fc251-45a8-41a3-8fcf-5855d7fe07da/ebdbfe46-9733-485c-9ca3-58f0449d57c1"
-					(reference "C149")
+					(reference "C120")
 					(unit 1)
 				)

Commit message: Annotations
Parts:
- renumbered C117 to C130, C118 to C131, C119 to C132, C120 to C133, C121 to C134, C122 to C135, C123 to C136, C124 to C137, C125 to C138, R45 to R48
Changed lines of the file:
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@@
 		(on_board yes)
 		(dnp no)
-		(property "Reference" "C121"
+		(property "Reference" "C134"
 			(at 221.742 88.3855 0)
 			(effects
@@
 			(project "srad-camera"
 				(path "/da62c771-e8c9-451f-8df1-ec995aadcb11/279fc251-45a8-41a3-8fcf-5855d7fe07da/ebdbfe46-9733-485c-9ca3-58f0449d57c1"
-					(reference "C121")
+					(reference "C134")
 					(unit 1)
 				)
@@
 		(dnp no)
 		(fields_autoplaced yes)
-		(property "Reference" "#PWR087"
+		(property "Reference" "#PWR097"
 			(at 88.9 107.95 0)
 			(effects
@@
 			(project "srad-camera"
 				(path "/da62c771-e8c9-451f-8df1-ec995aadcb11/279fc251-45a8-41a3-8fcf-5855d7fe07da/ebdbfe46-9733-485c-9ca3-58f0449d57c1"
-					(reference "#PWR087")
+					(reference "#PWR097")
 					(unit 1)
 				)
@@
 		(dnp no)
 		(fields_autoplaced yes)
-		(property "Reference" "#PWR081"
+		(property "Reference" "#PWR091"
 			(at 152.4 33.02 0)
 			(effects
@@
 			(project "srad-camera"
 				(path "/da62c771-e8c9-451f-8df1-ec995aadcb11/279fc251-45a8-41a3-8fcf-5855d7fe07da/ebdbfe46-9733-485c-9ca3-58f0449d57c1"
-					(reference "#PWR081")
+					(reference "#PWR091")
 					(unit 1)
 				)
@@
 		(on_board yes)
 		(dnp no)
-		(property "Reference" "#PWR089"
+		(property "Reference" "#PWR099"
 			(at 96.52 137.16 0)
 			(effects
@@
 			(project "srad-camera"
 				(path "/da62c771-e8c9-451f-8df1-ec995aadcb11/279fc251-45a8-41a3-8fcf-5855d7fe07da/ebdbfe46-9733-485c-9ca3-58f0449d57c1"
-					(reference "#PWR089")
+					(reference "#PWR099")
 					(unit 1)
 				)
@@
 		(dnp no)
 		(fields_autoplaced yes)
-		(property "Reference" "#PWR086"
+		(property "Reference" "#PWR096"
 			(at 91.44 92.71 0)
 			(effects
@@
 			(project "srad-camera"
 				(path "/da62c771-e8c9-451f-8df1-ec995aadcb11/279fc251-45a8-41a3-8fcf-5855d7fe07da/ebdbfe46-9733-485c-9ca3-58f0449d57c1"
-					(reference "#PWR086")
+					(reference "#PWR096")
 					(unit 1)
 				)
@@
 		(on_board yes)
 		(dnp no)
-		(property "Reference" "#PWR084"
+		(property "Reference" "#PWR094"
 			(at 224.79 77.47 0)
 			(effects
@@
 			(project "srad-camera"
 				(path "/da62c771-e8c9-451f-8df1-ec995aadcb11/279fc251-45a8-41a3-8fcf-5855d7fe07da/ebdbfe46-9733-485c-9ca3-58f0449d57c1"
-					(reference "#PWR084")
+					(reference "#PWR094")
 					(unit 1)
 				)
@@
 		(on_board yes)
 		(dnp no)
-		(property "Reference" "#PWR083"
+		(property "Reference" "#PWR093"
 			(at 219.71 60.96 0)
 			(effects
@@
 			(project "srad-camera"
 				(path "/da62c771-e8c9-451f-8df1-ec995aadcb11/279fc251-45a8-41a3-8fcf-5855d7fe07da/ebdbfe46-9733-485c-9ca3-58f0449d57c1"
-					(reference "#PWR083")
+					(reference "#PWR093")
 					(unit 1)
 				)
@@
 		(on_board yes)
 		(dnp no)
-		(property "Reference" "C125"
+		(property "Reference" "C138"
 			(at 94.488 126.238 0)
 			(effects
@@
 			(project "srad-camera"
 				(path "/da62c771-e8c9-451f-8df1-ec995aadcb11/279fc251-45a8-41a3-8fcf-5855d7fe07da/ebdbfe46-9733-485c-9ca3-58f0449d57c1"
-					(reference "C125")
+					(reference "C138")
 					(unit 1)
 				)
@@
 		(on_board yes)
 		(dnp no)
-		(property "Reference" "C118"
+		(property "Reference" "C131"
 			(at 213.868 66.548 0)
 			(effects
@@
 			(project "srad-camera"
 				(path "/da62c771-e8c9-451f-8df1-ec995aadcb11/279fc251-45a8-41a3-8fcf-5855d7fe07da/ebdbfe46-9733-485c-9ca3-58f0449d57c1"
-					(reference "C118")
+					(reference "C131")
 					(unit 1)
 				)
@@
 		(dnp no)
 		(fields_autoplaced yes)
-		(property "Reference" "#PWR082"
+		(property "Reference" "#PWR092"
 			(at 148.59 46.99 0)
 			(effects
@@
 			(project "srad-camera"
 				(path "/da62c771-e8c9-451f-8df1-ec995aadcb11/279fc251-45a8-41a3-8fcf-5855d7fe07da/ebdbfe46-9733-485c-9ca3-58f0449d57c1"
-					(reference "#PWR082")
+					(reference "#PWR092")
 					(unit 1)
 				)
@@
 		(on_board yes)
 		(dnp no)
-		(property "Reference" "C124"
+		(property "Reference" "C137"
 			(at 210.312 124.968 0)
 			(effects
@@
 			(project "srad-camera"
 				(path "/da62c771-e8c9-451f-8df1-ec995aadcb11/279fc251-45a8-41a3-8fcf-5855d7fe07da/ebdbfe46-9733-485c-9ca3-58f0449d57c1"
-					(reference "C124")
+					(reference "C137")
 					(unit 1)
 				)
@@
 		(on_board yes)
 		(dnp no)
-		(property "Reference" "#PWR088"
+		(property "Reference" "#PWR098"
 			(at 208.28 135.89 0)
 			(effects
@@
 			(project "srad-camera"
 				(path "/da62c771-e8c9-451f-8df1-ec995aadcb11/279fc251-45a8-41a3-8fcf-5855d7fe07da/ebdbfe46-9733-485c-9ca3-58f0449d57c1"
-					(reference "#PWR088")
+					(reference "#PWR098")
 					(unit 1)
 				)
@@
 		(on_board yes)
 		(dnp no)
-		(property "Reference" "#PWR085"
+		(property "Reference" "#PWR095"
 			(at 219.71 91.44 0)
 			(effects
@@
 			(project "srad-camera"
 				(path "/da62c771-e8c9-451f-8df1-ec995aadcb11/279fc251-45a8-41a3-8fcf-5855d7fe07da/ebdbfe46-9733-485c-9ca3-58f0449d57c1"
-					(reference "#PWR085")
+					(reference "#PWR095")
 					(unit 1)
 				)
@@
 		(dnp no)
 		(fields_autoplaced yes)
-		(property "Reference" "C123"
+		(property "Reference" "C136"
 			(at 94.488 95.758 0)
 			(effects
@@
 			(project "srad-camera"
 				(path "/da62c771-e8c9-451f-8df1-ec995aadcb11/279fc251-45a8-41a3-8fcf-5855d7fe07da/ebdbfe46-9733-485c-9ca3-58f0449d57c1"
-					(reference "C123")
+					(reference "C136")
 					(unit 1)
 				)
@@
 		(dnp no)
 		(fields_autoplaced yes)
-		(property "Reference" "C122"
+		(property "Reference" "C135"
 			(at 87.122 95.758 0)
 			(effects
@@
 			(project "srad-camera"
 				(path "/da62c771-e8c9-451f-8df1-ec995aadcb11/279fc251-45a8-41a3-8fcf-5855d7fe07da/ebdbfe46-9733-485c-9ca3-58f0449d57c1"
-					(reference "C122")
+					(reference "C135")
 					(unit 1)
 				)
@@
 		(on_board yes)
 		(dnp no)
-		(property "Reference" "C119"
+		(property "Reference" "C132"
 			(at 221.742 66.5545 0)
 			(effects
@@
 			(project "srad-camera"
 				(path "/da62c771-e8c9-451f-8df1-ec995aadcb11/279fc251-45a8-41a3-8fcf-5855d7fe07da/ebdbfe46-9733-485c-9ca3-58f0449d57c1"
-					(reference "C119")
+					(reference "C132")
 					(unit 1)
 				)
@@
 		(on_board yes)
 		(dnp no)
-		(property "Reference" "R45"
+		(property "Reference" "R48"
 			(at 152.4 35.4767 90)
 			(effects
@@
 			(project "srad-camera"
 				(path "/da62c771-e8c9-451f-8df1-ec995aadcb11/279fc251-45a8-41a3-8fcf-5855d7fe07da/ebdbfe46-9733-485c-9ca3-58f0449d57c1"
-					(reference "R45")
+					(reference "R48")
 					(unit 1)
 				)
@@
 		(dnp no)
 		(fields_autoplaced yes)
-		(property "Reference" "C117"
+		(property "Reference" "C130"
 			(at 146.266 35.6114 0)
 			(effects
@@
 			(project "srad-camera"
 				(path "/da62c771-e8c9-451f-8df1-ec995aadcb11/279fc251-45a8-41a3-8fcf-5855d7fe07da/ebdbfe46-9733-485c-9ca3-58f0449d57c1"
-					(reference "C117")
+					(reference "C130")
 					(unit 1)
 				)
@@
 		(on_board yes)
 		(dnp no)
-		(property "Reference" "C120"
+		(property "Reference" "C133"
 			(at 213.868 88.392 0)
 			(effects
@@
 			(project "srad-camera"
 				(path "/da62c771-e8c9-451f-8df1-ec995aadcb11/279fc251-45a8-41a3-8fcf-5855d7fe07da/ebdbfe46-9733-485c-9ca3-58f0449d57c1"
-					(reference "C120")
+					(reference "C133")
 					(unit 1)
 				)

Commit message: Minor tweaks + annotations
Other:
- moved on the sheet: R48
Changed lines of the file:
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@@
 	(wire
 		(pts
-			(xy 156.21 33.02) (xy 154.94 33.02)
+			(xy 160.02 33.02) (xy 157.48 33.02)
 		)
 		(stroke
@@
 	(wire
 		(pts
-			(xy 148.59 33.02) (xy 149.86 33.02)
+			(xy 148.59 33.02) (xy 152.4 33.02)
 		)
 		(stroke
@@
 	(wire
 		(pts
-			(xy 147.32 33.02) (xy 148.59 33.02)
+			(xy 139.7 33.02) (xy 148.59 33.02)
 		)
 		(stroke
@@
 	(hierarchical_label "VCCA_1V8_IMG"
 		(shape input)
-		(at 147.32 33.02 180)
+		(at 139.7 33.02 180)
 		(effects
 			(font
@@
 	(symbol
 		(lib_id "power:VCC")
-		(at 156.21 33.02 270)
+		(at 160.02 33.02 270)
 		(unit 1)
 		(exclude_from_sim no)
@@
 		(fields_autoplaced yes)
 		(property "Reference" "#PWR091"
-			(at 152.4 33.02 0)
+			(at 156.21 33.02 0)
 			(effects
 				(font
@@
 		)
 		(property "Value" "MIPI_AVDD_1V8"
-			(at 166.5417 33.02 90)
+			(at 170.3517 33.02 90)
 			(effects
 				(font
@@
 		)
 		(property "Footprint" ""
-			(at 156.21 33.02 0)
+			(at 160.02 33.02 0)
 			(effects
 				(font
@@
 		)
 		(property "Datasheet" ""
-			(at 156.21 33.02 0)
+			(at 160.02 33.02 0)
 			(effects
 				(font
@@
 		)
 		(property "Description" "Power symbol creates a global label with name \"VCC\""
-			(at 156.21 33.02 0)
+			(at 160.02 33.02 0)
 			(effects
 				(font
@@
 	(symbol
 		(lib_id "Device:R_Small")
-		(at 152.4 33.02 270)
+		(at 154.94 33.02 270)
 		(unit 1)
 		(exclude_from_sim no)
@@
 		(dnp no)
 		(property "Reference" "R48"
-			(at 152.4 35.4767 90)
+			(at 154.94 35.4767 90)
 			(effects
 				(font
@@
 		)
 		(property "Value" "1R"
-			(at 152.4 37.338 90)
+			(at 154.94 37.338 90)
 			(effects
 				(font
@@
 		)
 		(property "Footprint" ""
-			(at 152.4 33.02 0)
+			(at 154.94 33.02 0)
 			(effects
 				(font
@@
 		)
 		(property "Datasheet" "~"
-			(at 152.4 33.02 0)
+			(at 154.94 33.02 0)
 			(effects
 				(font
@@
 		)
 		(property "Description" "Resistor, small symbol"
-			(at 152.4 33.02 0)
+			(at 154.94 33.02 0)
 			(effects
 				(font
@@
 		)
 		(property "ADDITIONAL CARD DETECTION PINS" ""
-			(at 152.4 33.02 0)
+			(at 154.94 33.02 0)
 			(effects
 				(font
@@
 		)
 		(property "CARD CONNECTION MODE" ""
-			(at 152.4 33.02 0)
+			(at 154.94 33.02 0)
 			(effects
 				(font
@@
 		)
 		(property "CARD TYPE" ""
-			(at 152.4 33.02 0)
+			(at 154.94 33.02 0)
 			(effects
 				(font
@@
 		)
 		(property "CONNECTOR TYPE" ""
-			(at 152.4 33.02 0)
+			(at 154.94 33.02 0)
 			(effects
 				(font
@@
 		)
 		(property "SUPPLEMENTARY FEATURES" ""
-			(at 152.4 33.02 0)
+			(at 154.94 33.02 0)
 			(effects
 				(font

Commit message: Start on PCB design
Parts:
- C128: renamed from C130; footprint (none) -> Capacitor_SMD:C_0603_1608Metric; LCSC PART NAME (none) -> C15849
- C129: renamed from C131; footprint (none) -> Capacitor_SMD:C_0402_1005Metric; LCSC PART NAME (none) -> C1525
- C130: renamed from C132; footprint (none) -> Capacitor_SMD:C_0402_1005Metric; LCSC PART NAME (none) -> C1525
- C131: renamed from C133; footprint (none) -> Capacitor_SMD:C_0402_1005Metric; LCSC PART NAME (none) -> C1525
- C132: renamed from C134; footprint (none) -> Capacitor_SMD:C_0402_1005Metric; LCSC PART NAME (none) -> C1525
- C133: renamed from C135; footprint (none) -> Capacitor_SMD:C_0402_1005Metric; LCSC PART NAME (none) -> C1525
- C134: renamed from C136; footprint (none) -> Capacitor_SMD:C_0402_1005Metric; LCSC PART NAME (none) -> C1525
- C135: renamed from C137; footprint (none) -> Capacitor_SMD:C_0402_1005Metric; LCSC PART NAME (none) -> C1525
- C136: renamed from C138; footprint (none) -> Capacitor_SMD:C_0402_1005Metric; LCSC PART NAME (none) -> C1525
- R49: renamed from R48; footprint (none) -> Resistor_SMD:R_0402_1005Metric; LCSC PART NAME (none) -> C25086
- U5: LCSC PART NAME RK3566 -> (none)
