File: kicad/subsheets/rk-domains/ddr-phy.kicad_sch (KiCad schematic)
At the start: 12 parts, among them U5 RK3566

Commit message: Mark as R1.0
Parts:
- renumbered C73 to C79, C74 to C80, C75 to C81, C76 to C82, C77 to C83, C78 to C84, C79 to C85, C80 to C86, C81 to C87, C82 to C88, R29 to R32
Other:
- company: (none) -> UVic Rocketry
Changed lines of the file:
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@@
 	(title_block
 		(title "DDR PHY")
+		(date "2025-11-23")
+		(rev "1.0")
+		(company "UVic Rocketry")
+		(comment 1 "Author: Eric Handley")
 	)
 	(text "Caps under\npackage"
@@
 		(dnp no)
 		(fields_autoplaced yes)
-		(property "Reference" "#PWR049"
+		(property "Reference" "#PWR060"
 			(at 204.47 133.35 0)
 			(effects
@@
 			(project "srad-camera"
 				(path "/da62c771-e8c9-451f-8df1-ec995aadcb11/279fc251-45a8-41a3-8fcf-5855d7fe07da/b02e9bc7-ee33-4919-a384-9a6d4f12bf5d"
-					(reference "#PWR049")
+					(reference "#PWR060")
 					(unit 1)
 				)
@@
 		(dnp no)
 		(fields_autoplaced yes)
-		(property "Reference" "#PWR051"
+		(property "Reference" "#PWR062"
 			(at 118.11 157.48 0)
 			(effects
@@
 			(project "srad-camera"
 				(path "/da62c771-e8c9-451f-8df1-ec995aadcb11/279fc251-45a8-41a3-8fcf-5855d7fe07da/b02e9bc7-ee33-4919-a384-9a6d4f12bf5d"
-					(reference "#PWR051")
+					(reference "#PWR062")
 					(unit 1)
 				)
@@
 		(dnp no)
 		(fields_autoplaced yes)
-		(property "Reference" "#PWR046"
+		(property "Reference" "#PWR059"
 			(at 193.04 113.03 0)
 			(effects
@@
 			(project "srad-camera"
 				(path "/da62c771-e8c9-451f-8df1-ec995aadcb11/279fc251-45a8-41a3-8fcf-5855d7fe07da/b02e9bc7-ee33-4919-a384-9a6d4f12bf5d"
-					(reference "#PWR046")
+					(reference "#PWR059")
 					(unit 1)
 				)
@@
 		(dnp no)
 		(fields_autoplaced yes)
-		(property "Reference" "#PWR050"
+		(property "Reference" "#PWR061"
 			(at 204.47 153.67 0)
 			(effects
@@
 			(project "srad-camera"
 				(path "/da62c771-e8c9-451f-8df1-ec995aadcb11/279fc251-45a8-41a3-8fcf-5855d7fe07da/b02e9bc7-ee33-4919-a384-9a6d4f12bf5d"
-					(reference "#PWR050")
+					(reference "#PWR061")
 					(unit 1)
 				)
@@
 		(dnp no)
 		(fields_autoplaced yes)
-		(property "Reference" "C73"
+		(property "Reference" "C79"
 			(at 172.72 127.254 0)
 			(effects
@@
 			(project "srad-camera"
 				(path "/da62c771-e8c9-451f-8df1-ec995aadcb11/279fc251-45a8-41a3-8fcf-5855d7fe07da/b02e9bc7-ee33-4919-a384-9a6d4f12bf5d"
-					(reference "C73")
+					(reference "C79")
 					(unit 1)
 				)
@@
 		(dnp no)
 		(fields_autoplaced yes)
-		(property "Reference" "C81"
+		(property "Reference" "C87"
 			(at 193.04 147.574 0)
 			(effects
@@
 			(project "srad-camera"
 				(path "/da62c771-e8c9-451f-8df1-ec995aadcb11/279fc251-45a8-41a3-8fcf-5855d7fe07da/b02e9bc7-ee33-4919-a384-9a6d4f12bf5d"
-					(reference "C81")
+					(reference "C87")
 					(unit 1)
 				)
@@
 		(dnp no)
 		(fields_autoplaced yes)
-		(property "Reference" "C80"
+		(property "Reference" "C86"
 			(at 185.42 147.574 0)
 			(effects
@@
 			(project "srad-camera"
 				(path "/da62c771-e8c9-451f-8df1-ec995aadcb11/279fc251-45a8-41a3-8fcf-5855d7fe07da/b02e9bc7-ee33-4919-a384-9a6d4f12bf5d"
-					(reference "C80")
+					(reference "C86")
 					(unit 1)
 				)
@@
 		(dnp no)
 		(fields_autoplaced yes)
-		(property "Reference" "R29"
+		(property "Reference" "R32"
 			(at 182.88 108.1489 90)
 			(effects
@@
 			(project "srad-camera"
 				(path "/da62c771-e8c9-451f-8df1-ec995aadcb11/279fc251-45a8-41a3-8fcf-5855d7fe07da/b02e9bc7-ee33-4919-a384-9a6d4f12bf5d"
-					(reference "R29")
+					(reference "R32")
 					(unit 1)
 				)
@@
 		(dnp no)
 		(fields_autoplaced yes)
-		(property "Reference" "C77"
+		(property "Reference" "C83"
 			(at 199.39 127.254 0)
 			(effects
@@
 			(project "srad-camera"
 				(path "/da62c771-e8c9-451f-8df1-ec995aadcb11/279fc251-45a8-41a3-8fcf-5855d7fe07da/b02e9bc7-ee33-4919-a384-9a6d4f12bf5d"
-					(reference "C77")
+					(reference "C83")
 					(unit 1)
 				)
@@
 		(dnp no)
 		(fields_autoplaced yes)
-		(property "Reference" "C78"
+		(property "Reference" "C84"
 			(at 172.72 147.574 0)
 			(effects
@@
 			(project "srad-camera"
 				(path "/da62c771-e8c9-451f-8df1-ec995aadcb11/279fc251-45a8-41a3-8fcf-5855d7fe07da/b02e9bc7-ee33-4919-a384-9a6d4f12bf5d"
-					(reference "C78")
+					(reference "C84")
 					(unit 1)
 				)
@@
 		(dnp no)
 		(fields_autoplaced yes)
-		(property "Reference" "C79"
+		(property "Reference" "C85"
 			(at 179.07 147.574 0)
 			(effects
@@
 			(project "srad-camera"
 				(path "/da62c771-e8c9-451f-8df1-ec995aadcb11/279fc251-45a8-41a3-8fcf-5855d7fe07da/b02e9bc7-ee33-4919-a384-9a6d4f12bf5d"
-					(reference "C79")
+					(reference "C85")
 					(unit 1)
 				)
@@
 		(dnp no)
 		(fields_autoplaced yes)
-		(property "Reference" "C76"
+		(property "Reference" "C82"
 			(at 193.04 127.254 0)
 			(effects
@@
 			(project "srad-camera"
 				(path "/da62c771-e8c9-451f-8df1-ec995aadcb11/279fc251-45a8-41a3-8fcf-5855d7fe07da/b02e9bc7-ee33-4919-a384-9a6d4f12bf5d"
-					(reference "C76")
+					(reference "C82")
 					(unit 1)
 				)
@@
 		(dnp no)
 		(fields_autoplaced yes)
-		(property "Reference" "C74"
+		(property "Reference" "C80"
 			(at 179.07 127.254 0)
 			(effects
@@
 			(project "srad-camera"
 				(path "/da62c771-e8c9-451f-8df1-ec995aadcb11/279fc251-45a8-41a3-8fcf-5855d7fe07da/b02e9bc7-ee33-4919-a384-9a6d4f12bf5d"
-					(reference "C74")
+					(reference "C80")
 					(unit 1)
 				)
@@
 		(dnp no)
 		(fields_autoplaced yes)
-		(property "Reference" "C75"
+		(property "Reference" "C81"
 			(at 185.42 127.254 0)
 			(effects
@@
 			(project "srad-camera"
 				(path "/da62c771-e8c9-451f-8df1-ec995aadcb11/279fc251-45a8-41a3-8fcf-5855d7fe07da/b02e9bc7-ee33-4919-a384-9a6d4f12bf5d"
-					(reference "C75")
+					(reference "C81")
 					(unit 1)
 				)
@@
 		(dnp no)
 		(fields_autoplaced yes)
-		(property "Reference" "C82"
+		(property "Reference" "C88"
 			(at 199.39 147.574 0)
 			(effects
@@
 			(project "srad-camera"
 				(path "/da62c771-e8c9-451f-8df1-ec995aadcb11/279fc251-45a8-41a3-8fcf-5855d7fe07da/b02e9bc7-ee33-4919-a384-9a6d4f12bf5d"
-					(reference "C82")
+					(reference "C88")
 					(unit 1)
 				)

Commit message: Annotations
Parts:
- renumbered C87 to C100, C88 to C101, C79 to C92, C80 to C93, C81 to C94, C82 to C95, C83 to C96, C84 to C97, C85 to C98, C86 to C99, R32 to R35
Changed lines of the file:
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@@
 		(dnp no)
 		(fields_autoplaced yes)
-		(property "Reference" "#PWR060"
+		(property "Reference" "#PWR070"
 			(at 204.47 133.35 0)
 			(effects
@@
 			(project "srad-camera"
 				(path "/da62c771-e8c9-451f-8df1-ec995aadcb11/279fc251-45a8-41a3-8fcf-5855d7fe07da/b02e9bc7-ee33-4919-a384-9a6d4f12bf5d"
-					(reference "#PWR060")
+					(reference "#PWR070")
 					(unit 1)
 				)
@@
 		(dnp no)
 		(fields_autoplaced yes)
-		(property "Reference" "#PWR062"
+		(property "Reference" "#PWR072"
 			(at 118.11 157.48 0)
 			(effects
@@
 			(project "srad-camera"
 				(path "/da62c771-e8c9-451f-8df1-ec995aadcb11/279fc251-45a8-41a3-8fcf-5855d7fe07da/b02e9bc7-ee33-4919-a384-9a6d4f12bf5d"
-					(reference "#PWR062")
+					(reference "#PWR072")
 					(unit 1)
 				)
@@
 		(dnp no)
 		(fields_autoplaced yes)
-		(property "Reference" "#PWR059"
+		(property "Reference" "#PWR069"
 			(at 193.04 113.03 0)
 			(effects
@@
 			(project "srad-camera"
 				(path "/da62c771-e8c9-451f-8df1-ec995aadcb11/279fc251-45a8-41a3-8fcf-5855d7fe07da/b02e9bc7-ee33-4919-a384-9a6d4f12bf5d"
-					(reference "#PWR059")
+					(reference "#PWR069")
 					(unit 1)
 				)
@@
 		(dnp no)
 		(fields_autoplaced yes)
-		(property "Reference" "#PWR061"
+		(property "Reference" "#PWR071"
 			(at 204.47 153.67 0)
 			(effects
@@
 			(project "srad-camera"
 				(path "/da62c771-e8c9-451f-8df1-ec995aadcb11/279fc251-45a8-41a3-8fcf-5855d7fe07da/b02e9bc7-ee33-4919-a384-9a6d4f12bf5d"
-					(reference "#PWR061")
+					(reference "#PWR071")
 					(unit 1)
 				)
@@
 		(dnp no)
 		(fields_autoplaced yes)
-		(property "Reference" "C79"
+		(property "Reference" "C92"
 			(at 172.72 127.254 0)
 			(effects
@@
 			(project "srad-camera"
 				(path "/da62c771-e8c9-451f-8df1-ec995aadcb11/279fc251-45a8-41a3-8fcf-5855d7fe07da/b02e9bc7-ee33-4919-a384-9a6d4f12bf5d"
-					(reference "C79")
+					(reference "C92")
 					(unit 1)
 				)
@@
 		(dnp no)
 		(fields_autoplaced yes)
-		(property "Reference" "C87"
+		(property "Reference" "C100"
 			(at 193.04 147.574 0)
 			(effects
@@
 			(project "srad-camera"
 				(path "/da62c771-e8c9-451f-8df1-ec995aadcb11/279fc251-45a8-41a3-8fcf-5855d7fe07da/b02e9bc7-ee33-4919-a384-9a6d4f12bf5d"
-					(reference "C87")
+					(reference "C100")
 					(unit 1)
 				)
@@
 		(dnp no)
 		(fields_autoplaced yes)
-		(property "Reference" "C86"
+		(property "Reference" "C99"
 			(at 185.42 147.574 0)
 			(effects
@@
 			(project "srad-camera"
 				(path "/da62c771-e8c9-451f-8df1-ec995aadcb11/279fc251-45a8-41a3-8fcf-5855d7fe07da/b02e9bc7-ee33-4919-a384-9a6d4f12bf5d"
-					(reference "C86")
+					(reference "C99")
 					(unit 1)
 				)
@@
 		(dnp no)
 		(fields_autoplaced yes)
-		(property "Reference" "R32"
+		(property "Reference" "R35"
 			(at 182.88 108.1489 90)
 			(effects
@@
 			(project "srad-camera"
 				(path "/da62c771-e8c9-451f-8df1-ec995aadcb11/279fc251-45a8-41a3-8fcf-5855d7fe07da/b02e9bc7-ee33-4919-a384-9a6d4f12bf5d"
-					(reference "R32")
+					(reference "R35")
 					(unit 1)
 				)
@@
 		(dnp no)
 		(fields_autoplaced yes)
-		(property "Reference" "C83"
+		(property "Reference" "C96"
 			(at 199.39 127.254 0)
 			(effects
@@
 			(project "srad-camera"
 				(path "/da62c771-e8c9-451f-8df1-ec995aadcb11/279fc251-45a8-41a3-8fcf-5855d7fe07da/b02e9bc7-ee33-4919-a384-9a6d4f12bf5d"
-					(reference "C83")
+					(reference "C96")
 					(unit 1)
 				)
@@
 		(dnp no)
 		(fields_autoplaced yes)
-		(property "Reference" "C84"
+		(property "Reference" "C97"
 			(at 172.72 147.574 0)
 			(effects
@@
 			(project "srad-camera"
 				(path "/da62c771-e8c9-451f-8df1-ec995aadcb11/279fc251-45a8-41a3-8fcf-5855d7fe07da/b02e9bc7-ee33-4919-a384-9a6d4f12bf5d"
-					(reference "C84")
+					(reference "C97")
 					(unit 1)
 				)
@@
 		(dnp no)
 		(fields_autoplaced yes)
-		(property "Reference" "C85"
+		(property "Reference" "C98"
 			(at 179.07 147.574 0)
 			(effects
@@
 			(project "srad-camera"
 				(path "/da62c771-e8c9-451f-8df1-ec995aadcb11/279fc251-45a8-41a3-8fcf-5855d7fe07da/b02e9bc7-ee33-4919-a384-9a6d4f12bf5d"
-					(reference "C85")
+					(reference "C98")
 					(unit 1)
 				)
@@
 		(dnp no)
 		(fields_autoplaced yes)
-		(property "Reference" "C82"
+		(property "Reference" "C95"
 			(at 193.04 127.254 0)
 			(effects
@@
 			(project "srad-camera"
 				(path "/da62c771-e8c9-451f-8df1-ec995aadcb11/279fc251-45a8-41a3-8fcf-5855d7fe07da/b02e9bc7-ee33-4919-a384-9a6d4f12bf5d"
-					(reference "C82")
+					(reference "C95")
 					(unit 1)
 				)
@@
 		(dnp no)
 		(fields_autoplaced yes)
-		(property "Reference" "C80"
+		(property "Reference" "C93"
 			(at 179.07 127.254 0)
 			(effects
@@
 			(project "srad-camera"
 				(path "/da62c771-e8c9-451f-8df1-ec995aadcb11/279fc251-45a8-41a3-8fcf-5855d7fe07da/b02e9bc7-ee33-4919-a384-9a6d4f12bf5d"
-					(reference "C80")
+					(reference "C93")
 					(unit 1)
 				)
@@
 		(dnp no)
 		(fields_autoplaced yes)
-		(property "Reference" "C81"
+		(property "Reference" "C94"
 			(at 185.42 127.254 0)
 			(effects
@@
 			(project "srad-camera"
 				(path "/da62c771-e8c9-451f-8df1-ec995aadcb11/279fc251-45a8-41a3-8fcf-5855d7fe07da/b02e9bc7-ee33-4919-a384-9a6d4f12bf5d"
-					(reference "C81")
+					(reference "C94")
 					(unit 1)
 				)
@@
 		(dnp no)
 		(fields_autoplaced yes)
-		(property "Reference" "C88"
+		(property "Reference" "C101"
 			(at 199.39 147.574 0)
 			(effects
@@
 			(project "srad-camera"
 				(path "/da62c771-e8c9-451f-8df1-ec995aadcb11/279fc251-45a8-41a3-8fcf-5855d7fe07da/b02e9bc7-ee33-4919-a384-9a6d4f12bf5d"
-					(reference "C88")
+					(reference "C101")
 					(unit 1)
 				)

Commit message: Start on PCB design
Parts:
- C90: renamed from C92; footprint (none) -> Capacitor_SMD:C_0402_1005Metric; LCSC PART NAME (none) -> C1525
- C91: renamed from C93; footprint (none) -> Capacitor_SMD:C_0402_1005Metric; LCSC PART NAME (none) -> C1525
- C92: renamed from C94; footprint (none) -> Capacitor_SMD:C_0402_1005Metric; LCSC PART NAME (none) -> C1525
- C93: renamed from C95; footprint (none) -> Capacitor_SMD:C_0805_2012Metric; LCSC PART NAME (none) -> C1779
- C94: renamed from C96; footprint (none) -> Capacitor_SMD:C_0805_2012Metric; LCSC PART NAME (none) -> C1779
- C95: renamed from C97; footprint (none) -> Capacitor_SMD:C_0402_1005Metric; LCSC PART NAME (none) -> C1525
- C96: renamed from C98; footprint (none) -> Capacitor_SMD:C_0402_1005Metric; LCSC PART NAME (none) -> C1525
- C97: renamed from C99; footprint (none) -> Capacitor_SMD:C_0402_1005Metric; LCSC PART NAME (none) -> C1525
- C98: renamed from C100; footprint (none) -> Capacitor_SMD:C_0805_2012Metric; LCSC PART NAME (none) -> C1779
- C99: renamed from C101; footprint (none) -> Capacitor_SMD:C_0805_2012Metric; LCSC PART NAME (none) -> C1779
- R36: renamed from R35; value 120R 1% -> 120R; footprint (none) -> Resistor_SMD:R_0402_1005Metric; LCSC PART NAME (none) -> C25079
- U5: LCSC PART NAME RK3566 -> (none)
Changed lines of the file:
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@@
 			)
 		)
-		(property "LCSC PART NAME" "RK3566"
+		(property "LCSC PART NAME" ""
 			(at 202.692 95.25 0)
 			(effects
@@
 		(dnp no)
 		(fields_autoplaced yes)
-		(property "Reference" "C92"
+		(property "Reference" "C90"
 			(at 172.72 127.254 0)
 			(effects
@@
 			)
 		)
-		(property "Footprint" ""
+		(property "Footprint" "Capacitor_SMD:C_0402_1005Metric"
 			(at 172.72 121.92 0)
 			(effects
@@
 			)
 		)
-		(property "V" ""
-			(at 172.72 121.92 90)
+		(property "LCSC PART NAME" "C1525"
+			(at 172.72 121.92 0)
 			(effects
 				(font
@@
 			(project "srad-camera"
 				(path "/da62c771-e8c9-451f-8df1-ec995aadcb11/279fc251-45a8-41a3-8fcf-5855d7fe07da/b02e9bc7-ee33-4919-a384-9a6d4f12bf5d"
-					(reference "C92")
+					(reference "C90")
 					(unit 1)
 				)
@@
 		(dnp no)
 		(fields_autoplaced yes)
-		(property "Reference" "C100"
+		(property "Reference" "C98"
 			(at 193.04 147.574 0)
 			(effects
@@
 			)
 		)
-		(property "Footprint" ""
+		(property "Footprint" "Capacitor_SMD:C_0805_2012Metric"
 			(at 193.04 142.24 0)
 			(effects
@@
 			)
 		)
-		(property "V" ""
-			(at 193.04 142.24 90)
+		(property "LCSC PART NAME" "C1779"
+			(at 193.04 142.24 0)
 			(effects
 				(font
@@
 			(project "srad-camera"
 				(path "/da62c771-e8c9-451f-8df1-ec995aadcb11/279fc251-45a8-41a3-8fcf-5855d7fe07da/b02e9bc7-ee33-4919-a384-9a6d4f12bf5d"
-					(reference "C100")
+					(reference "C98")
 					(unit 1)
 				)
@@
 		(dnp no)
 		(fields_autoplaced yes)
-		(property "Reference" "C99"
+		(property "Reference" "C97"
 			(at 185.42 147.574 0)
 			(effects
@@
 			)
 		)
-		(property "Footprint" ""
+		(property "Footprint" "Capacitor_SMD:C_0402_1005Metric"
 			(at 185.42 142.24 0)
 			(effects
@@
 			)
 		)
-		(property "V" ""
-			(at 185.42 142.24 90)
-			(effects
-				(font
-					(size 1.27 1.27)
-				)
-				(hide yes)
-			)
-		)
 		(property "ADDITIONAL CARD DETECTION PINS" ""
 			(at 185.42 142.24 90)
@@
 		(property "SUPPLEMENTARY FEATURES" ""
 			(at 185.42 142.24 90)
+			(effects
+				(font
+					(size 1.27 1.27)
+				)
+				(hide yes)
+			)
+		)
+		(property "LCSC PART NAME" "C1525"
+			(at 185.42 142.24 0)
 			(effects
 				(font
@@
 			(project "srad-camera"
 				(path "/da62c771-e8c9-451f-8df1-ec995aadcb11/279fc251-45a8-41a3-8fcf-5855d7fe07da/b02e9bc7-ee33-4919-a384-9a6d4f12bf5d"
-					(reference "C99")
+					(reference "C97")
 					(unit 1)
 				)
@@
 		(dnp no)
 		(fields_autoplaced yes)
-		(property "Reference" "R35"
+		(property "Reference" "R36"
 			(at 182.88 108.1489 90)
 			(effects
@@
 			)
 		)
-		(property "Value" "120R 1%"
+		(property "Value" "120R"
 			(at 182.88 110.5732 90)
 			(effects
@@
 			)
 		)
-		(property "Footprint" ""
+		(property "Footprint" "Resistor_SMD:R_0402_1005Metric"
 			(at 182.88 113.03 0)
 			(effects
@@
 		)
 		(property "SUPPLEMENTARY FEATURES" ""
+			(at 182.88 113.03 90)
+			(effects
+				(font
+					(size 1.27 1.27)
+				)
+				(hide yes)
+			)
+		)
+		(property "LCSC PART NAME" "C25079"
 			(at 182.88 113.03 90)
 			(effects
@@
 			(project "srad-camera"
 				(path "/da62c771-e8c9-451f-8df1-ec995aadcb11/279fc251-45a8-41a3-8fcf-5855d7fe07da/b02e9bc7-ee33-4919-a384-9a6d4f12bf5d"
-					(reference "R35")
+					(reference "R36")
 					(unit 1)
 				)
@@
 		(dnp no)
 		(fields_autoplaced yes)
-		(property "Reference" "C96"
+		(property "Reference" "C94"
 			(at 199.39 127.254 0)
 			(effects
@@
 			)
 		)
-		(property "Footprint" ""
+		(property "Footprint" "Capacitor_SMD:C_0805_2012Metric"
 			(at 199.39 121.92 0)
 			(effects
@@
 			)
 		)
-		(property "V" ""
-			(at 199.39 121.92 90)
+		(property "LCSC PART NAME" "C1779"
+			(at 199.39 121.92 0)
 			(effects
 				(font
@@
 			(project "srad-camera"
 				(path "/da62c771-e8c9-451f-8df1-ec995aadcb11/279fc251-45a8-41a3-8fcf-5855d7fe07da/b02e9bc7-ee33-4919-a384-9a6d4f12bf5d"
-					(reference "C96")
+					(reference "C94")
 					(unit 1)
 				)
@@
 		(dnp no)
 		(fields_autoplaced yes)
-		(property "Reference" "C97"
+		(property "Reference" "C95"
 			(at 172.72 147.574 0)
 			(effects
@@
 			)
 		)
-		(property "Footprint" ""
+		(property "Footprint" "Capacitor_SMD:C_0402_1005Metric"
 			(at 172.72 142.24 0)
 			(effects
@@
 			)
 		)
-		(property "V" ""
-			(at 172.72 142.24 90)
+		(property "LCSC PART NAME" "C1525"
+			(at 172.72 142.24 0)
 			(effects
 				(font
@@
 			(project "srad-camera"
 				(path "/da62c771-e8c9-451f-8df1-ec995aadcb11/279fc251-45a8-41a3-8fcf-5855d7fe07da/b02e9bc7-ee33-4919-a384-9a6d4f12bf5d"
-					(reference "C97")
+					(reference "C95")
 					(unit 1)
 				)
@@
 		(dnp no)
 		(fields_autoplaced yes)
-		(property "Reference" "C98"
+		(property "Reference" "C96"
 			(at 179.07 147.574 0)
 			(effects
@@
 			)
 		)
-		(property "Footprint" ""
+		(property "Footprint" "Capacitor_SMD:C_0402_1005Metric"
 			(at 179.07 142.24 0)
 			(effects
@@
 			)
 		)
-		(property "V" ""
-			(at 179.07 142.24 90)
+		(property "LCSC PART NAME" "C1525"
+			(at 179.07 142.24 0)
 			(effects
 				(font
@@
 			(project "srad-camera"
 				(path "/da62c771-e8c9-451f-8df1-ec995aadcb11/279fc251-45a8-41a3-8fcf-5855d7fe07da/b02e9bc7-ee33-4919-a384-9a6d4f12bf5d"
-					(reference "C98")
+					(reference "C96")
 					(unit 1)
 				)
@@
 		(dnp no)
 		(fields_autoplaced yes)
-		(property "Reference" "C95"
+		(property "Reference" "C93"
 			(at 193.04 127.254 0)
 			(effects
@@
 			)
 		)
-		(property "Footprint" ""
+		(property "Footprint" "Capacitor_SMD:C_0805_2012Metric"
 			(at 193.04 121.92 0)
 			(effects
@@
 			)
 		)
-		(property "V" ""
-			(at 193.04 121.92 90)
+		(property "LCSC PART NAME" "C1779"
+			(at 193.04 121.92 0)
 			(effects
 				(font
@@
 			(project "srad-camera"
 				(path "/da62c771-e8c9-451f-8df1-ec995aadcb11/279fc251-45a8-41a3-8fcf-5855d7fe07da/b02e9bc7-ee33-4919-a384-9a6d4f12bf5d"
-					(reference "C95")
+					(reference "C93")
 					(unit 1)
 				)
@@
 		(dnp no)
 		(fields_autoplaced yes)
-		(property "Reference" "C93"
+		(property "Reference" "C91"
 			(at 179.07 127.254 0)
 			(effects
@@
 			)
 		)
-		(property "Footprint" ""
+		(property "Footprint" "Capacitor_SMD:C_0402_1005Metric"
 			(at 179.07 121.92 0)
 			(effects
@@
 			)
 		)
-		(property "V" ""
-			(at 179.07 121.92 90)
+		(property "LCSC PART NAME" "C1525"
+			(at 179.07 121.92 0)
 			(effects
 				(font
@@
 			(project "srad-camera"
 				(path "/da62c771-e8c9-451f-8df1-ec995aadcb11/279fc251-45a8-41a3-8fcf-5855d7fe07da/b02e9bc7-ee33-4919-a384-9a6d4f12bf5d"
-					(reference "C93")
+					(reference "C91")
 					(unit 1)
 				)
@@
 		(dnp no)
 		(fields_autoplaced yes)
-		(property "Reference" "C94"
+		(property "Reference" "C92"
 			(at 185.42 127.254 0)
 			(effects
@@
 			)
 		)
-		(property "Footprint" ""
+		(property "Footprint" "Capacitor_SMD:C_0402_1005Metric"
 			(at 185.42 121.92 0)
 			(effects
@@
 			)
 		)
-		(property "V" ""
-			(at 185.42 121.92 90)
-			(effects
-				(font
-					(size 1.27 1.27)
-				)
-				(hide yes)
-			)
-		)
 		(property "ADDITIONAL CARD DETECTION PINS" ""
 			(at 185.42 121.92 90)
@@
 		(property "SUPPLEMENTARY FEATURES" ""
 			(at 185.42 121.92 90)
+			(effects
+				(font
+					(size 1.27 1.27)
+				)
+				(hide yes)
+			)
+		)
+		(property "LCSC PART NAME" "C1525"
+			(at 185.42 121.92 0)
 			(effects
 				(font
@@
 			(project "srad-camera"
 				(path "/da62c771-e8c9-451f-8df1-ec995aadcb11/279fc251-45a8-41a3-8fcf-5855d7fe07da/b02e9bc7-ee33-4919-a384-9a6d4f12bf5d"
-					(reference "C94")
+					(reference "C92")
 					(unit 1)
 				)
@@
 		(dnp no)
 		(fields_autoplaced yes)
-		(property "Reference" "C101"
+		(property "Reference" "C99"
 			(at 199.39 147.574 0)
 			(effects
@@
 			)
 		)
-		(property "Footprint" ""
+		(property "Footprint" "Capacitor_SMD:C_0805_2012Metric"
 			(at 199.39 142.24 0)
 			(effects
@@
 			)
 		)
-		(property "V" ""
-			(at 199.39 142.24 90)
+		(property "LCSC PART NAME" "C1779"
+			(at 199.39 142.24 0)
 			(effects
 				(font
@@
 			(project "srad-camera"
 				(path "/da62c771-e8c9-451f-8df1-ec995aadcb11/279fc251-45a8-41a3-8fcf-5855d7fe07da/b02e9bc7-ee33-4919-a384-9a6d4f12bf5d"
-					(reference "C101")
+					(reference "C99")
 					(unit 1)
 				)
