File: kicad/subsheets/rk-domains/ddr-phy.kicad_sch (KiCad schematic)
At the start: 12 parts, among them U5 RK3566

Commit message: Remove power/decoupling for unused power domains
Parts:
- renumbered C90 to C88, C91 to C89, C92 to C90, C93 to C91, C94 to C92, C95 to C93, C96 to C94, C97 to C95, C98 to C96, C99 to C97
Changed lines of the file:
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@@
 		(dnp no)
 		(fields_autoplaced yes)
-		(property "Reference" "#PWR070"
+		(property "Reference" "#PWR073"
 			(at 204.47 133.35 0)
 			(effects
@@
 			(project "srad-camera"
 				(path "/da62c771-e8c9-451f-8df1-ec995aadcb11/279fc251-45a8-41a3-8fcf-5855d7fe07da/b02e9bc7-ee33-4919-a384-9a6d4f12bf5d"
-					(reference "#PWR070")
+					(reference "#PWR073")
 					(unit 1)
 				)
@@
 		(dnp no)
 		(fields_autoplaced yes)
-		(property "Reference" "#PWR072"
+		(property "Reference" "#PWR075"
 			(at 118.11 157.48 0)
 			(effects
@@
 			(project "srad-camera"
 				(path "/da62c771-e8c9-451f-8df1-ec995aadcb11/279fc251-45a8-41a3-8fcf-5855d7fe07da/b02e9bc7-ee33-4919-a384-9a6d4f12bf5d"
-					(reference "#PWR072")
+					(reference "#PWR075")
 					(unit 1)
 				)
@@
 		(dnp no)
 		(fields_autoplaced yes)
-		(property "Reference" "#PWR069"
+		(property "Reference" "#PWR072"
 			(at 193.04 113.03 0)
 			(effects
@@
 			(project "srad-camera"
 				(path "/da62c771-e8c9-451f-8df1-ec995aadcb11/279fc251-45a8-41a3-8fcf-5855d7fe07da/b02e9bc7-ee33-4919-a384-9a6d4f12bf5d"
-					(reference "#PWR069")
+					(reference "#PWR072")
 					(unit 1)
 				)
@@
 		(dnp no)
 		(fields_autoplaced yes)
-		(property "Reference" "#PWR071"
+		(property "Reference" "#PWR074"
 			(at 204.47 153.67 0)
 			(effects
@@
 			(project "srad-camera"
 				(path "/da62c771-e8c9-451f-8df1-ec995aadcb11/279fc251-45a8-41a3-8fcf-5855d7fe07da/b02e9bc7-ee33-4919-a384-9a6d4f12bf5d"
-					(reference "#PWR071")
+					(reference "#PWR074")
 					(unit 1)
 				)
@@
 		(dnp no)
 		(fields_autoplaced yes)
-		(property "Reference" "C90"
+		(property "Reference" "C88"
 			(at 172.72 127.254 0)
 			(effects
@@
 			(project "srad-camera"
 				(path "/da62c771-e8c9-451f-8df1-ec995aadcb11/279fc251-45a8-41a3-8fcf-5855d7fe07da/b02e9bc7-ee33-4919-a384-9a6d4f12bf5d"
-					(reference "C90")
+					(reference "C88")
 					(unit 1)
 				)
@@
 		(dnp no)
 		(fields_autoplaced yes)
-		(property "Reference" "C98"
+		(property "Reference" "C96"
 			(at 193.04 147.574 0)
 			(effects
@@
 			(project "srad-camera"
 				(path "/da62c771-e8c9-451f-8df1-ec995aadcb11/279fc251-45a8-41a3-8fcf-5855d7fe07da/b02e9bc7-ee33-4919-a384-9a6d4f12bf5d"
-					(reference "C98")
+					(reference "C96")
 					(unit 1)
 				)
@@
 		(dnp no)
 		(fields_autoplaced yes)
-		(property "Reference" "C97"
+		(property "Reference" "C95"
 			(at 185.42 147.574 0)
 			(effects
@@
 			(project "srad-camera"
 				(path "/da62c771-e8c9-451f-8df1-ec995aadcb11/279fc251-45a8-41a3-8fcf-5855d7fe07da/b02e9bc7-ee33-4919-a384-9a6d4f12bf5d"
-					(reference "C97")
+					(reference "C95")
 					(unit 1)
 				)
@@
 		(dnp no)
 		(fields_autoplaced yes)
-		(property "Reference" "C94"
+		(property "Reference" "C92"
 			(at 199.39 127.254 0)
 			(effects
@@
 			(project "srad-camera"
 				(path "/da62c771-e8c9-451f-8df1-ec995aadcb11/279fc251-45a8-41a3-8fcf-5855d7fe07da/b02e9bc7-ee33-4919-a384-9a6d4f12bf5d"
-					(reference "C94")
+					(reference "C92")
 					(unit 1)
 				)
@@
 		(dnp no)
 		(fields_autoplaced yes)
-		(property "Reference" "C95"
+		(property "Reference" "C93"
 			(at 172.72 147.574 0)
 			(effects
@@
 			(project "srad-camera"
 				(path "/da62c771-e8c9-451f-8df1-ec995aadcb11/279fc251-45a8-41a3-8fcf-5855d7fe07da/b02e9bc7-ee33-4919-a384-9a6d4f12bf5d"
-					(reference "C95")
+					(reference "C93")
 					(unit 1)
 				)
@@
 		(dnp no)
 		(fields_autoplaced yes)
-		(property "Reference" "C96"
+		(property "Reference" "C94"
 			(at 179.07 147.574 0)
 			(effects
@@
 			(project "srad-camera"
 				(path "/da62c771-e8c9-451f-8df1-ec995aadcb11/279fc251-45a8-41a3-8fcf-5855d7fe07da/b02e9bc7-ee33-4919-a384-9a6d4f12bf5d"
-					(reference "C96")
+					(reference "C94")
 					(unit 1)
 				)
@@
 		(dnp no)
 		(fields_autoplaced yes)
-		(property "Reference" "C93"
+		(property "Reference" "C91"
 			(at 193.04 127.254 0)
 			(effects
@@
 			(project "srad-camera"
 				(path "/da62c771-e8c9-451f-8df1-ec995aadcb11/279fc251-45a8-41a3-8fcf-5855d7fe07da/b02e9bc7-ee33-4919-a384-9a6d4f12bf5d"
-					(reference "C93")
+					(reference "C91")
 					(unit 1)
 				)
@@
 		(dnp no)
 		(fields_autoplaced yes)
-		(property "Reference" "C91"
+		(property "Reference" "C89"
 			(at 179.07 127.254 0)
 			(effects
@@
 			(project "srad-camera"
 				(path "/da62c771-e8c9-451f-8df1-ec995aadcb11/279fc251-45a8-41a3-8fcf-5855d7fe07da/b02e9bc7-ee33-4919-a384-9a6d4f12bf5d"
-					(reference "C91")
+					(reference "C89")
 					(unit 1)
 				)
@@
 		(dnp no)
 		(fields_autoplaced yes)
-		(property "Reference" "C92"
+		(property "Reference" "C90"
 			(at 185.42 127.254 0)
 			(effects
@@
 			(project "srad-camera"
 				(path "/da62c771-e8c9-451f-8df1-ec995aadcb11/279fc251-45a8-41a3-8fcf-5855d7fe07da/b02e9bc7-ee33-4919-a384-9a6d4f12bf5d"
-					(reference "C92")
+					(reference "C90")
 					(unit 1)
 				)
@@
 		(dnp no)
 		(fields_autoplaced yes)
-		(property "Reference" "C99"
+		(property "Reference" "C97"
 			(at 199.39 147.574 0)
 			(effects
@@
 			(project "srad-camera"
 				(path "/da62c771-e8c9-451f-8df1-ec995aadcb11/279fc251-45a8-41a3-8fcf-5855d7fe07da/b02e9bc7-ee33-4919-a384-9a6d4f12bf5d"
-					(reference "C99")
+					(reference "C97")
 					(unit 1)
 				)

Commit message: All major components placed on board
Parts:
- C91, C92, C96, C97: footprint Capacitor_SMD:C_0805_2012Metric -> Capacitor_SMD:C_0402_1005Metric
Changed lines of the file:
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@@
 			)
 		)
-		(property "Footprint" "Capacitor_SMD:C_0805_2012Metric"
+		(property "Footprint" "Capacitor_SMD:C_0402_1005Metric"
 			(at 193.04 142.24 0)
 			(effects
@@
 			)
 		)
-		(property "Footprint" "Capacitor_SMD:C_0805_2012Metric"
+		(property "Footprint" "Capacitor_SMD:C_0402_1005Metric"
 			(at 199.39 121.92 0)
 			(effects
@@
 			)
 		)
-		(property "Footprint" "Capacitor_SMD:C_0805_2012Metric"
+		(property "Footprint" "Capacitor_SMD:C_0402_1005Metric"
 			(at 193.04 121.92 0)
 			(effects
@@
 			)
 		)
-		(property "Footprint" "Capacitor_SMD:C_0805_2012Metric"
+		(property "Footprint" "Capacitor_SMD:C_0402_1005Metric"
 			(at 199.39 142.24 0)
 			(effects
